File: hardware/kicad/dsp-regulator-hat-rev-b/DSP-Regulator-HAT-RevB.kicad_sch (KiCad schematic)
At the start: 213 parts, among them J1 FW-10-05-X-D-XXX-XXX-A, J10 1935161, J11 1935161, J12 20021121-00010C4LF, J13 Conn_02x05_Odd_Even, J16 Conn_01x01_Pin, J17 Conn_01x01_Pin, J18 Conn_01x01_Pin, J19 SWD_Debug_Header, J2 FW-10-05-X-D-XXX-XXX-A, J20 Connector, USB-TYPE-C-16P, J21 Display Uart, J3 Conn_01x01_Pin, J4 Conn_01x01_Pin, J5 Conn_01x01_Pin, J6 Conn_01x01_Pin, J7 Conn_01x01_Pin, J8 Conn_01x01_Pin, J9 1935161, Q1 PSMN5R2-60YL, Q10 PSMN5R2-60YL, Q11 PSMN5R2-60YL, Q12 PSMN5R2-60YL, Q2 PSMN5R2-60YL, Q3 PSMN5R2-60YL, Q4 PSMN5R2-60YL, Q5 PSMN5R2-60YL, Q6 PSMN5R2-60YL, Q7 PSMN5R2-60YL, Q8 PSMN5R2-60YL, Q9 PSMN5R2-60YL, U1 INA3221, U10 STM32_BLUE -, U11 W25Q128, U12 CH340C, U2 INA3221, U3 TLV1704AIPWR, U4 TLV1704AIPWR, U5 TLV1704AIPWR, U6 INA3221, U7 74HC595D, U8 74HC595D, U9 AMS1117-3.3

Commit message: hw(channel3): split J2 pin 06 to +V Adj Channel for CrowPanel 5V supply
- Split J2 pin 06 from +5V_Boot to dedicated +V Adj Channel net in
  both Rev-B schematics and netlists
- Reroute J21 pin 1 (CrowPanel display power) from +5V_Boot to
  +V Adj Channel in Rev-B HAT schematic and netlist
- PWR_FLAG at (123.19, 375.92) migrates to +V Adj Channel net via
  retained wire (374.65->375.92); J2 pins 08/10/12 remain on +5V_Boot
- DSP Regulator (PCB Rev-C prep): mark U8, R26, R43 as DNP;
  set R11=240 Ohm (lower FB->GND), R41=750 Ohm (future upper resistor)
- Update netlists manually to reflect schematic changes; re-export
  from KiCad GUI required for full ERC/DRC validation
- Connector contract: +V Adj Channel now PASS (was FAIL)

NOTE: R41 wire topology in DSP Regulator needs KiCad GUI edit to
connect as upper resistor (pin1->+V Adj Channel, pin2->FB).
VSENSE_ADJ+/-, ISET_MPU_Channel_3 failures are pre-existing.

Co-authored-by: Copilot <223556219+Copilot@users.noreply.github.com>
Parts:
- removed C10, C11, C27, C28, C30: 100nF, PCM_JLCPCB:C_0805, symbol PCM_JLCPCB-Capacitors:0805,100nF,(2)
- removed C18, C19: 1nF, PCM_JLCPCB:C_0805, symbol PCM_JLCPCB-Capacitors:0805,1nF
- removed C22, C4: 10uF, PCM_JLCPCB:C_0805, symbol PCM_JLCPCB-Capacitors:0805,10uF,(2)
- removed C24: C_Small_US, Capacitor_SMD:CP_Elec_10x10, symbol Device:C_Small_US
- removed D10: Green, PCM_JLCPCB:D_0805, symbol PCM_JLCPCB-Diodes:LED,0805,Green
- removed D6: 1N5819WS, Diode_SMD:D_SOD-323, symbol Diode:1N5819WS
- removed D7: SMBJ6.0CA, PCM_JLCPCB:D_SMB, symbol PCM_JLCPCB-Diodes:TVS-Bi,SMBJ6.0CA
- removed J11: 1935161, digikey-footprints:Terminal_Block_D1.3mm_P5mm, symbol dk_Terminal-Blocks-Wire-to-Board:1935161
- removed J3, J4: Conn_01x01_Pin, Connector_Wire:SolderWire-1sqmm_1x01_D1.4mm_OD2.7mm, symbol Connector:Conn_01x01_Pin
- removed L2: L_Ferrite, Inductor_SMD:L_1206_3216Metric, symbol Device:L_Ferrite
- removed POT5, POT6: 3296W-1-103LF, Potentiometer_THT:Potentiometer_Bourns_3296W_Vertical, symbol 1My_Basic components:3296W-1-103LF
- removed Q11, Q12, Q5, Q6: PSMN5R2-60YL, Package_TO_SOT_SMD:LFPAK56, symbol Transistor_FET:PSMN5R2-60YL
- removed R13, R14: 100Ω, PCM_JLCPCB:R_0805, symbol PCM_JLCPCB-Resistors:0805,100Ω
- removed R20, R21: R, Resistor_SMD:R_2512_6332Metric, symbol Device:R
- removed R30, R31, R32, R33, R59, R63, R64: 10Ω, PCM_JLCPCB:R_0805, symbol PCM_JLCPCB-Resistors:0805,10Ω
- removed R44, R47: 1kΩ, PCM_JLCPCB:R_0805, symbol PCM_JLCPCB-Resistors:0805,1kΩ
- removed R45, R46, R71: 10kΩ, PCM_JLCPCB:R_0805, symbol PCM_JLCPCB-Resistors:0805,10kΩ
- removed R5, R54, R6: 100kΩ, PCM_JLCPCB:R_0805, symbol PCM_JLCPCB-Resistors:0805,100kΩ
- removed R56: 270Ω, PCM_JLCPCB:R_0805, symbol PCM_JLCPCB-Resistors:0805,270Ω
- removed R67, R68, R69: 0Ω, PCM_JLCPCB:R_0805, symbol PCM_JLCPCB-Resistors:0805,0Ω
- removed TP10, TP5, TP6: TestPoint_Small, symbol Connector:TestPoint_Small
- removed unit 2 of U5
- removed unit 1 of U5
- removed U6: INA3221, Package_DFN_QFN:Texas_RGV0016A_VQFN-16-1EP_4x4mm_P0.65mm_EP2.1x2.1mm, symbol Power_Management:INA3221
- removed U8: 74HC595D, PCM_JLCPCB:SOIC-16_L9.9-W3.9-P1.27-LS6.0-BL, symbol PCM_JLCPCB-ICs:Shift Register, 1 In, 8 Out, 74HC595D,118
Connections:
- net Channel _3_High_range is gone; now on an unnamed net: U7.6 (Q6)
- net Channel _3_low_range is gone; now on net ISET_MPU_3V3: U7.5 (Q5)
- net +5V_Boot: now also J2.08, J2.10, J2.12; no longer J13.1 (Pin_1), J2.02
- net +V Adj Channel: now also J13.1 (Pin_1); no longer J2.08, J2.10, J2.12
- net GND: now also J2.02
- net ISET_MPU_3V3: no longer U7.7 (Q7)
- net ISET_MPU_Channel_3: no longer J1.13
- net at J12.3: now also U7.7 (Q7)
- net 3.3_Select: no longer names the net of J1.15
- net VSENSE_ADJ+: no longer names the net of D2.1
- net VSENSE_ADJ+: no longer J1.02
- net VSENSE_ADJ-: no longer names the net of J1.04
- net VSENSE_ADJ-: no longer D1.4
Other:
- moved on the sheet: J12
