File: hardware/kicad/dsp-regulator-hat-rev-b/DSP-Regulator-HAT-RevB.kicad_sch (KiCad schematic)
At the start: 213 parts, among them J1 FW-10-05-X-D-XXX-XXX-A, J10 1935161, J11 1935161, J12 20021121-00010C4LF, J13 Conn_02x05_Odd_Even, J16 Conn_01x01_Pin, J17 Conn_01x01_Pin, J18 Conn_01x01_Pin, J19 SWD_Debug_Header, J2 FW-10-05-X-D-XXX-XXX-A, J20 Connector, USB-TYPE-C-16P, J21 Display Uart, J3 Conn_01x01_Pin, J4 Conn_01x01_Pin, J5 Conn_01x01_Pin, J6 Conn_01x01_Pin, J7 Conn_01x01_Pin, J8 Conn_01x01_Pin, J9 1935161, Q1 PSMN5R2-60YL, Q10 PSMN5R2-60YL, Q11 PSMN5R2-60YL, Q12 PSMN5R2-60YL, Q2 PSMN5R2-60YL, Q3 PSMN5R2-60YL, Q4 PSMN5R2-60YL, Q5 PSMN5R2-60YL, Q6 PSMN5R2-60YL, Q7 PSMN5R2-60YL, Q8 PSMN5R2-60YL, Q9 PSMN5R2-60YL, U1 INA3221, U10 STM32_BLUE -, U11 W25Q128, U12 CH340C, U2 INA3221, U3 TLV1704AIPWR, U4 TLV1704AIPWR, U5 TLV1704AIPWR, U6 INA3221, U7 74HC595D, U8 74HC595D, U9 AMS1117-3.3

Commit message: Closeout handoff and checkpoint PCB/netlist updates
Parts:
- removed C10, C11, C27, C28, C30: 100nF, PCM_JLCPCB:C_0805, symbol PCM_JLCPCB-Capacitors:0805,100nF,(2)
- removed C18, C19: 1nF, PCM_JLCPCB:C_0805, symbol PCM_JLCPCB-Capacitors:0805,1nF
- removed C22, C4: 10uF, PCM_JLCPCB:C_0805, symbol PCM_JLCPCB-Capacitors:0805,10uF,(2)
- removed C24: C_Small_US, Capacitor_SMD:CP_Elec_10x10, symbol Device:C_Small_US
- removed D10: Green, PCM_JLCPCB:D_0805, symbol PCM_JLCPCB-Diodes:LED,0805,Green
- removed D6: 1N5819WS, Diode_SMD:D_SOD-323, symbol Diode:1N5819WS
- removed D7: SMBJ6.0CA, PCM_JLCPCB:D_SMB, symbol PCM_JLCPCB-Diodes:TVS-Bi,SMBJ6.0CA
- removed J11: 1935161, digikey-footprints:Terminal_Block_D1.3mm_P5mm, symbol dk_Terminal-Blocks-Wire-to-Board:1935161
- removed J3, J4: Conn_01x01_Pin, Connector_Wire:SolderWire-1sqmm_1x01_D1.4mm_OD2.7mm, symbol Connector:Conn_01x01_Pin
- removed L2: L_Ferrite, Inductor_SMD:L_1206_3216Metric, symbol Device:L_Ferrite
- removed POT5, POT6: 3296W-1-103LF, Potentiometer_THT:Potentiometer_Bourns_3296W_Vertical, symbol 1My_Basic components:3296W-1-103LF
- removed Q11, Q12, Q5, Q6: PSMN5R2-60YL, Package_TO_SOT_SMD:LFPAK56, symbol Transistor_FET:PSMN5R2-60YL
- removed R10, R15, R49, R50, R52, R67, R68, R69, R9: 0Ω, PCM_JLCPCB:R_0805, symbol PCM_JLCPCB-Resistors:0805,0Ω
- removed R13, R14: 100Ω, PCM_JLCPCB:R_0805, symbol PCM_JLCPCB-Resistors:0805,100Ω
- removed R20, R21: R, Resistor_SMD:R_2512_6332Metric, symbol Device:R
- removed R30, R31, R32, R33, R34, R35, R59, R63, R64: 10Ω, PCM_JLCPCB:R_0805, symbol PCM_JLCPCB-Resistors:0805,10Ω
- removed R44, R47: 1kΩ, PCM_JLCPCB:R_0805, symbol PCM_JLCPCB-Resistors:0805,1kΩ
- removed R45, R46, R71: 10kΩ, PCM_JLCPCB:R_0805, symbol PCM_JLCPCB-Resistors:0805,10kΩ
- removed R5, R54, R6: 100kΩ, PCM_JLCPCB:R_0805, symbol PCM_JLCPCB-Resistors:0805,100kΩ
- removed R56: 270Ω, PCM_JLCPCB:R_0805, symbol PCM_JLCPCB-Resistors:0805,270Ω
- removed TP10, TP5, TP6: TestPoint_Small, symbol Connector:TestPoint_Small
- removed U5: TLV1704AIPWR, Package_SO:TSSOP-14_4.4x5mm_P0.65mm, symbol 1My_IC's:TLV1704AIPWR
- removed U6: INA3221, Package_DFN_QFN:Texas_RGV0016A_VQFN-16-1EP_4x4mm_P0.65mm_EP2.1x2.1mm, symbol Power_Management:INA3221
- removed U8: 74HC595D, PCM_JLCPCB:SOIC-16_L9.9-W3.9-P1.27-LS6.0-BL, symbol PCM_JLCPCB-ICs:Shift Register, 1 In, 8 Out, 74HC595D,118
- added D6: Yellow, PCM_JLCPCB:D_0805, symbol PCM_JLCPCB-Diodes_1:LED,0805,Yellow
- added D7: US1M, Diode_SMD:D_SMA, symbol Diode:US1M
- added J11: USB Hub I2C, 1My_Parts_ Connectors:JST_B4B-XH-A, symbol 1My_Connectors:B4B-XH-A
- added J3: 20021121-00010C4LF, digikey-footprints:PinHeader_2x5_P1.27mm, symbol 1My_Basic components:20021121-00010C4LF
- added J4: Fan Control, digikey-footprints:PinHeader_1x2_P2.5mm_Drill1.1mm, symbol dk_Rectangular-Connectors-Headers-Male-Pins:B2B-XH-A_LF__SN_
- added Q5: AO3400A, PCM_JLCPCB:Q_SOT-23, symbol PCM_JLCPCB-Transistors_1:NMOS,AO3400A
- added R10: 100kΩ, PCM_JLCPCB:R_0805, symbol PCM_JLCPCB-Resistors:0805,100kΩ
- added R5: 270Ω, PCM_JLCPCB:R_0805, symbol PCM_JLCPCB-Resistors:0805,270Ω
- added R9: 100Ω, PCM_JLCPCB:R_0805, symbol PCM_JLCPCB-Resistors:0805,100Ω
- added U5: AHT20_C2757850, 1My_Parts_ ICs:Humidity sensor, symbol easyeda2kicad:AHT20_C2757850
- C23, C25: value C_Small_US -> 470uf
- D3, D4: LCSC (none) -> C191023
- H1, H2, H3, H4: footprint MountingHole:MountingHole_3.2mm_M3_Pad -> MountingHole:MountingHole_3.5mm_Pad_Via
- J12: LCSC (none) -> C41376037
- J13: value Conn_02x05_Odd_Even -> SWD_Debug_Header; LCSC (none) -> C53207560
- J19: LCSC (none) -> C53207560
- POT1, POT2, POT3, POT4: LCSC (none) -> C49190453
- R16: value R -> 20m ohms; LCSC C7420022 -> C49164694
- R17: value R -> 200m ohms
- R18: value R -> 20mΩ; LCSC C7420022 -> C49164694
- R19: value R -> 200mΩ
- TP1, TP13, TP14, TP2, TP3, TP4, TP7, TP8, TP9: footprint (none) -> Connector_PinHeader_1.00mm:PinHeader_1x01_P1.00mm_Vertical
- TP11, TP2_+5V1, TP_+3.3V1: LCSC (none) -> C5199798
- U9: LCSC (none) -> C6186
Connections:
- net +V Adj Channel is gone; now on net +5V_Boot: J2.06, J2.08, J2.10, J2.12
- net 3.3_Select is gone; now on net ISET_MPU_3V3: J1.15
- net Channel _3_low_range is gone; now on net ISET_MPU_3V3: U7.5 (Q5)
- net +3.3V Boot: now also U2.5 (A0), J11.1, J3.1, U5.2 (VDD)
- net +5V_Boot: now also J13.2 (Pin_2), D7.1 (K), J4.2; no longer J13.1 (Pin_1), J2.02
- net GND: now also J1.07, J1.09, J1.11, J1.13, J13.1 (Pin_1), J13.7 (Pin_7), J2.02, U1.5 (A0), J11.4, J3.10, J3.2, Q5.2 (S), R10.2, R5.2, U5.5 (GND); no longer J13.2 (Pin_2), J13.8 (Pin_8)
- net ISET_MPU_3V3: no longer J1.11, U7.7 (Q7)
- net ISET_MPU_5V: now also J1.05; no longer J1.07
- net Incoming (+): now also U2.2 (IN+3)
- net Incoming (-): now also U2.1 (IN-3)
- net I²C SCL_0: now also J11.2, J3.5, U5.3 (SCL)
- net I²C SDA_0: now also J11.3, J3.6, U5.4 (SDA)
- net NRST: now also J3.9
- net PB5: now also R9.1
- net PB6: now also J12.10; no longer J12.8
- net SWDCLK: now also J3.8
- net SWDIO: now also J3.7
- net UART1_RX: now also J3.4
- net UART1_TX: now also J3.3
- net VSENSE_3V3+: now also R58.2
- net VSENSE_5V+: no longer R58.2
- net B13: now reaches U10.2 (B13)
- net B13: now also J12.5
- net B14: now reaches U10.3 (B14)
- net B14: now also J12.1
- net Fan out: now reaches U10.34 (B1)
- net B15: now reaches U10.4 (B15)
- net B15: now also J12.9
- net at R80.1: now also J13.4 (Pin_4); no longer J13.3 (Pin_3)
- net at R86.2: now also J13.9 (Pin_9); no longer J13.10 (Pin_10)
- net at R77.2: now also J13.5 (Pin_5); no longer J13.6 (Pin_6)
- net at R73.2: now also J13.3 (Pin_3); no longer J13.4 (Pin_4)
- net at R81.1: now also J13.6 (Pin_6); no longer J13.5 (Pin_5)
- net at R82.1: now also J13.8 (Pin_8); no longer J13.7 (Pin_7)
- net at R83.1: now also J13.10 (Pin_10); no longer J13.9 (Pin_9)
- net Channel _3_High_range: no longer names the net of U7.6 (Q6)
- net ISET_MPU_Channel_3: no longer names the net of U10.27 (A2)
- net ISET_MPU_Channel_3: no longer J1.13
- net VSENSE_ADJ+: no longer names the net of D2.1
- net VSENSE_ADJ+: no longer J1.02
- net VSENSE_ADJ-: no longer names the net of J1.04
- net VSENSE_ADJ-: no longer D1.4
- new net: D7.2 (A), J4.1, Q5.3 (D)
- new net: Q5.1 (G), R10.1, R9.2
- new net: D6.1, R5.1
- new net: D6.2, U7.7 (Q7)
- no-connect marks 44 -> 43
Other:
- note added: "Logic analyzer connector"
- note removed: "Channel 3 Selectable"
- moved on the sheet: C12, C13, C26, C29, C3, C31, C32, C33, C34, C35, C36, C37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

Commit message: Finalize Rev-B pre-fab review
Parts:
- U10: footprint Module:Maple_Mini -> 1My_Parts_ MPUs:STM32 Blue
Connections:
- net Fan out: no longer names the net of U10.34 (B1)
- no-connect marks 43 -> 44
Other:
- note added: "Temp sensor"
Changed lines of the file:
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@@
 		)
 	)
+	(text "Temp sensor\n"
+		(exclude_from_sim no)
+		(at 197.358 273.304 0)
+		(effects
+			(font
+				(size 1.27 1.27)
+			)
+		)
+	)
 	(text "3.3v control"
 		(exclude_from_sim no)
@@
 	)
 	(junction
+		(at 121.92 187.96)
+		(diameter 0)
+		(color 0 0 0 0)
+	)
+	(junction
 		(at 50.8 153.67)
 		(diameter 0)
@@
 	)
 	(junction
-		(at 121.92 187.96)
-		(diameter 0)
-		(color 0 0 0 0)
-	)
-	(junction
 		(at 471.17 349.25)
 		(diameter 0)
@@
 	)
 	(no_connect
+		(at 219.71 203.2)
+	)
+	(no_connect
 		(at 219.71 220.98)
 	)
@@
 	(wire
 		(pts
-			(xy 121.92 181.61) (xy 121.92 187.96)
+			(xy 120.65 181.61) (xy 120.65 187.96)
 		)
 		(stroke
@@
 	(wire
 		(pts
+			(xy 121.92 187.96) (xy 127 187.96)
+		)
+		(stroke
+			(width 0)
+			(type default)
+		)
+	)
+	(wire
+		(pts
 			(xy 73.66 63.5) (xy 72.39 63.5)
 		)
@@
 	(wire
 		(pts
-			(xy 121.92 187.96) (xy 127 187.96)
-		)
-		(stroke
-			(width 0)
-			(type default)
-		)
-	)
-	(wire
-		(pts
 			(xy 97.79 339.09) (xy 97.79 341.63)
 		)
@@
 	(wire
 		(pts
-			(xy 111.76 181.61) (xy 121.92 181.61)
+			(xy 111.76 181.61) (xy 120.65 181.61)
 		)
 		(stroke
@@
 	(wire
 		(pts
+			(xy 120.65 187.96) (xy 121.92 187.96)
+		)
+		(stroke
+			(width 0)
+			(type default)
+		)
+	)
+	(wire
+		(pts
 			(xy 30.48 132.08) (xy 31.75 132.08)
 		)
@@
 		)
 	)
-	(global_label "Fan out"
-		(shape input)
-		(at 219.71 203.2 0)
-		(fields_autoplaced yes)
-		(effects
-			(font
-				(size 0.635 0.635)
-			)
-			(justify left)
-		)
-		(property "Intersheetrefs" "${INTERSHEET_REFS}"
-			(at 224.8917 203.2 0)
-			(effects
-				(font
-					(size 1.27 1.27)
-				)
-				(justify left)
-				(hide yes)
-			)
-		)
-	)
 	(global_label "VSENSE_3V3-"
 		(shape input)
@@
 			)
 		)
-		(property "Footprint" "Module:Maple_Mini"
+		(property "Footprint" "1My_Parts_ MPUs:STM32 Blue"
 			(at 168.91 167.64 0)
 			(effects
