File: hardware/kicad/dsp-regulator-hat-rev-b/DSP-Regulator-HAT-RevB.kicad_sch (KiCad schematic)
At the start: 163 parts, among them J1 FW-10-05-X-D-XXX-XXX-A, J10 1935161, J11 USB Hub I2C, J12 20021121-00010C4LF, J13 SWD_Debug_Header, J16 Conn_01x01_Pin, J17 Conn_01x01_Pin, J18 Conn_01x01_Pin, J19 SWD_Debug_Header, J2 FW-10-05-X-D-XXX-XXX-A, J20 Connector, USB-TYPE-C-16P, J21 Display Uart, J3 20021121-00010C4LF, J4 Fan Control, J5 Conn_01x01_Pin, J6 Conn_01x01_Pin, J7 Conn_01x01_Pin, J8 Conn_01x01_Pin, J9 1935161, Q1 PSMN5R2-60YL, Q10 PSMN5R2-60YL, Q2 PSMN5R2-60YL, Q3 PSMN5R2-60YL, Q4 PSMN5R2-60YL, Q5 AO3400A, Q7 PSMN5R2-60YL, Q8 PSMN5R2-60YL, Q9 PSMN5R2-60YL, U1 INA3221, U10 STM32_BLUE -, U11 W25Q128, U12 CH340C, U2 INA3221, U3 TLV1704AIPWR, U4 TLV1704AIPWR, U5 AHT20_C2757850, U7 74HC595D, U9 AMS1117-3.3

Commit message: Capture VSENSE selector issue, SPICE validation, and pre-RevC routing blocker
Parts:
- removed R11, R12, R7, R8: 100Ω, PCM_JLCPCB:R_0805, symbol PCM_JLCPCB-Resistors:0805,100Ω
- removed R2: 100kΩ, PCM_JLCPCB:R_0805, symbol PCM_JLCPCB-Resistors:0805,100kΩ
- added C10, C11, C18, C19, C22, C24, C27, C4: 100nF, PCM_JLCPCB:C_0805, symbol PCM_JLCPCB-Capacitors:0805,100nF,(2)
- added D10, D14, D15, D16: 1SMA4742A, PCM_JLCPCB:D_DO-214AC(SMA), symbol PCM_JLCPCB-Diodes:Zener,1SMA4742A
- added R13, R30, R32, R8: 390kΩ, PCM_JLCPCB:R_0805, symbol PCM_JLCPCB-Resistors:0805,390kΩ
- added R14, R15, R31, R33, R7: 100kΩ, PCM_JLCPCB:R_0805, symbol PCM_JLCPCB-Resistors:0805,100kΩ
- added R2, R20, R21, R6: 10Ω, PCM_JLCPCB:R_0805, symbol PCM_JLCPCB-Resistors:0805,10Ω
- added U13, U14, U6, U8: LM74502HDDFR, Package_TO_SOT_SMD:Texas_DDF0008A_SOT-8_1.6x2.9mm_P0.65mm, symbol 1My_IC's:LM74502HDDFR
- 5mm1: value ~ -> (none)
- D2: now not fitted
- Q8: Manufacturer_Name Infineon -> (none); Manufacturer_Part_Number IRLZ44NPBF -> (none); Part HL3400 -> (none)
- U5: footprint 1My_Parts_ ICs:Humidity sensor -> Package_SON:WSON-6-1EP_3x3mm_P0.95mm; symbol easyeda2kicad:AHT20_C2757850 -> 1My_IC's:AHT20; Availability (none) -> Not in stock; Check_prices (none) -> https://www.snapeda.com/parts/AHT20/Asair/view-part/?ref=eda; Description_1 (none) -> Temperature and Humidity sensor; MANUFACTURER (none) -> Asair; MAXIMUM_PACKAGE_HEIGHT (none) -> 1.1mm; MF (none) -> Asair; MP (none) -> AHT20; PARTREV (none) -> V1.0; Package (none) -> Package; Price (none) -> None; STANDARD (none) -> IPC 7351B; SnapEDA_Link (none) -> https://www.snapeda.com/parts/AHT20/Asair/view-part/?ref=sn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
Connections:
- net +3.3V_Reg: now also Q1.5 (D), Q2.5 (D); no longer Q1.1 (S), Q1.2 (S), Q1.3 (S), Q2.1 (S), Q2.2 (S), Q2.3 (S)
- net +5V_Boot: now also C10.2, C11.1, C18.2, C19.1, C22.1, C24.2, C27.2, C4.1, R13.1, R30.1, R32.1, R8.1, U13.5 (VS), U14.5 (VS), U6.5 (VS), U8.5 (VS)
- net +5V_reg: now also Q3.5 (D), Q4.5 (D); no longer Q3.1 (S), Q3.2 (S), Q3.3 (S), Q4.1 (S), Q4.2 (S), Q4.3 (S)
- net ESP- GPIO 3.3V High: now also U6.1 (EN_UVLO)
- net ESP- GPIO 3.3V Low: now also U8.1 (EN_UVLO)
- net ESP- GPIO 5V Hi: now also U13.1 (EN_UVLO)
- net ESP- GPIO 5V Low: now also U14.1 (EN_UVLO)
- net GND: now also C10.1, C18.1, C24.1, C27.1, R14.2, R15.2, R31.2, R33.2, U13.2 (GND), U14.2 (GND), U6.2 (GND), U8.2 (GND); no longer R1.2, R3.2, R4.2
- net at C7.1, R16.1, R22.1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: now also Q7.5 (D); no longer Q7.1 (S), Q7.2 (S), Q7.3 (S)
- net Gate _3.3_HIGH: now reaches Q1.4 (G), Q7.4 (G)
- net Gate _3.3_HIGH: now also R1.2, D10.2 (cathode), R6.2; no longer R1.1
- net at C9.1, R18.1, R26.1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: now also Q9.5 (D); no longer Q9.1 (S), Q9.2 (S), Q9.3 (S)
- net Gate _5_High: now reaches Q3.4 (G), Q9.4 (G)
- net Gate _5_High: now also R4.2, D16.2 (cathode), R20.2; no longer R3.1
- net Gate _5_LOW: now reaches Q10.4 (G), Q4.4 (G)
- net Gate _5_LOW: now also R3.2, D15.2 (cathode), R21.2; no longer R4.1
- net at Q10.5 (D): now also C6.2, R19.1, R29.1, R43.1; no longer Q4.5 (D)
- net at C8.2, R17.1, R25.1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: now also Q8.5 (D); no longer Q8.1 (S), Q8.2 (S), Q8.3 (S)
- net Gate _3.3_LOW: now reaches Q2.4 (G), Q8.4 (G)
- net Gate _3.3_LOW: now also D14.2 (cathode), R2.2, R7.2
- net at U5.1 (NC): now also U5.6 (NC)
- new net: C19.2, U13.4 (VCAP)
- new net: R2.1, U8.6 (GATE)
- new net: R32.2, R33.1, U14.7 (OV)
- new net: C4.2, U6.4 (VCAP)
- new net: R21.1, U14.6 (GATE)
- new net: R20.1, U13.6 (GATE)
- new net: R15.1, R8.2, U8.7 (OV)
- new net: C22.2, U14.4 (VCAP)
- new net: R30.2, R31.1, U13.7 (OV)
- new net: C11.2, U8.4 (VCAP)
- new net: R6.1, U6.6 (GATE)
- new net: R13.2, R14.1, U6.7 (OV)
- new net SRC 3.3_HIGH: D10.1 (anode), Q1.1 (S), Q1.2 (S), Q1.3 (S), Q7.1 (S), Q7.2 (S), Q7.3 (S), R1.1, U6.8 (SRC)
- new net SRC 3.3_LOW: D14.1 (anode), Q2.1 (S), Q2.2 (S), Q2.3 (S), Q8.1 (S), Q8.2 (S), Q8.3 (S), R7.1, U8.8 (SRC)
- new net SRC 5_HIGH: D16.1 (anode), Q3.1 (S), Q3.2 (S), Q3.3 (S), Q9.1 (S), Q9.2 (S), Q9.3 (S), R4.1, U13.8 (SRC)
- new net SRC 5_LOW: D15.1 (anode), Q10.1 (S), Q10.2 (S), Q10.3 (S), Q4.1 (S), Q4.2 (S), Q4.3 (S), R3.1, U14.8 (SRC)
- no-connect marks 44 -> 47
Other:
- moved on the sheet: C1, C14, C15, C16, C17, C2, C20, C21, C23, C25, C6, C7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
