File: hardware/kicad/dsp-regulator-hat-rev-b/DSP-Regulator-HAT-RevB.kicad_pcb (KiCad board)
At the start: 2 copper layers, 100 x 102.6 mm, 163 parts, among them J1 FW-10-05-X-D-XXX-XXX-A, J10 1935161, J11 USB Hub I2C, J12 20021121-00010C4LF, J13 SWD_Debug_Header, J16 Conn_01x01_Pin, J17 Conn_01x01_Pin, J18 Conn_01x01_Pin, J19 SWD_Debug_Header, J2 FW-10-05-X-D-XXX-XXX-A, J20 Connector, USB-TYPE-C-16P, J21 Display Uart, J3 20021121-00010C4LF, J4 Fan Control, J5 Conn_01x01_Pin, J6 Conn_01x01_Pin, J7 Conn_01x01_Pin, J8 Conn_01x01_Pin, J9 1935161, Q1 PSMN5R2-60YL, Q10 PSMN5R2-60YL, Q2 PSMN5R2-60YL, Q3 PSMN5R2-60YL, Q4 PSMN5R2-60YL, Q5 AO3400A, Q7 PSMN5R2-60YL, Q8 PSMN5R2-60YL, Q9 PSMN5R2-60YL, U1 INA3221, U10 STM32_BLUE -, U11 W25Q128, U12 CH340C, U2 INA3221, U3 TLV1704AIPWR, U4 TLV1704AIPWR, U5 AHT20_C2757850, U7 74HC595D, U9 AMS1117-3.3

Commit message: Finalize Rev-B pre-fab review
Parts:
- U10: footprint Module:Maple_Mini -> 1My_Parts_ MPUs:STM32 Blue
- moved H3 0.42 mm to (92.8, 139.4)
- moved J13 0.36 mm to (138.3, 50.8)
- moved H1 0.30 mm to (92.8, 47.6)
Connections:
- U10 pad 34: Fan out -> unconnected-(U10-B1-Pad34)
Routing:
- net Net-(J13-Pin_6): track 7.51 -> 14.0 mm
- net +5V_Boot: track 272.4 -> 267.7 mm
- net Net-(J13-Pin_4): track 7.87 -> 11.7 mm
- net Net-(J13-Pin_8): track 5.73 -> 9.06 mm
- net Net-(J13-Pin_10): track 5.93 -> 8.87 mm
- net Net-(J13-Pin_9): track 14.6 -> 12.0 mm
- net Net-(J13-Pin_5): track 9.76 -> 7.42 mm
- net Net-(J13-Pin_3): track 12.4 -> 10.1 mm
- net Status_LED: track 65.5 -> 64.0 mm
- net SWDCLK: track 48.8 -> 48.0 mm
Other:
- board text added: "SPI HB"
- board text added: "SWDCLK"
- board text added: "SWDIO"
