File: hardware/kicad/usb-hub-next-iter/USB Hub Next Iter.kicad_sch (KiCad schematic)
At the start: 82 parts, among them J1 USB_A, J10 Connector, USB-TYPE-C-16P, J2 Connector, USB-TYPE-C-16P, J3 USB_A, J4 USB_A, J5 Connector, USB-TYPE-C- vert, J6 USB_A, J7 From 12V supply, J8 B5B-XH-A_LF__SN_, J9 B5B-XH-A_LF__SN_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

Commit message: usb-hub next-iter: add PWR_FLAGs and clear power-pin ERC issues
Parts:
- U3: symbol PCM_JLCPCB-Power:DC-DC, Buck, 4-40VIN, 3A, 5VOUT, (1) -> 1My_IC's:LM2576SX_-_Buck,_4-40VIN,_3A,_5VOUT,_(1)

Commit message: Closeout handoff and checkpoint PCB/netlist updates
Parts:
- added J11: STM32_SWD_BRIDGE_OUT, symbol Connector:Conn_01x05_Pin
- added R27, R28: 33Ω, PCM_JLCPCB:R_0805, symbol PCM_JLCPCB-Resistors:0805,33Ω
- added R29, R30: 0Ω, PCM_JLCPCB:R_1206, symbol PCM_JLCPCB-Resistors:1206,0Ω
Connections:
- net 3v3: now also J11.1 (Pin_1)
- net GND: now also J11.5 (Pin_5)
- net USB_BRIDGE_VBUS_SENSE: now reaches J10.A9B4 (VBUS), J10.B9A4 (VBUS), R21.1, R22.1, R23.1, U9.2 (IN-)
- net Port 2_D+ renamed USB_BRIDGE_DM
- net USB_BRIDGE_DM: now also U7.3 (-D1_2), R30.2; no longer U7.2 (+D1_2)
- net Port 2_D- renamed USB_BRIDGE_DP
- net USB_BRIDGE_DP: now also U7.2 (+D1_2), R29.1; no longer U7.3 (-D1_2)
- new net: J11.3 (Pin_3), R28.1
- new net: J11.2 (Pin_2), R27.1
- new net NRST_BRIDGE_OUT: J11.4 (Pin_4)
- new net SWDCLK_BRIDGE_OUT: R28.2, R30.1
- new net SWDIO_BRIDGE_OUT: R27.2, R29.2
- no-connect marks 11 -> 12
Other:
- moved on the sheet: R23
