File: hardware/kicad/dsp-regulator-rev-b/DSP-Regulator-RevB.kicad_sch (KiCad schematic)
At the start: 97 parts, among them J1 CLP-110-02-X-D, J2 CLP-110-02-X-D, J3 1935161, J4 Wire con, J5 Wire con, Q1 BSS138, Q16 BSS138, Q3 BSS138, Q4 BSS138, U2 LM2596S-ADJ, U3 LM2596S-ADJ, U4 LM2596S-ADJ, U5 LMV358IDR, U6 LMV358IDR

Commit message: Add 2026-08-10 handoff and capture STM32/board debug state
Parts:
- R25: now not fitted
Changed lines of the file:
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@@
 		(in_bom yes)
 		(on_board yes)
-		(dnp no)
+		(dnp yes)
 		(property "Reference" "R25"
 			(at 220.98 116.332 0)

Commit message: Capture VSENSE selector issue, SPICE validation, and pre-RevC routing blocker
Parts:
- 10mm1, 10mm2, 5mm1: value ~ -> (none)
- R25: now fitted
- R27, R28: now not fitted
Connections:
- net +12V: now also U5.8 (VCC+)
- net +5V_Boot: no longer U5.8 (VCC+)
