File: hardware/kicad/dsp-regulator-rev-c/DSP-Regulator-RevC.kicad_pcb (KiCad board)
At the start: 2 copper layers, 100 x 100 mm, 97 parts, among them J1 CLP-110-02-X-D, J2 CLP-110-02-X-D, J3 1935161, J4 Wire con, J5 Wire con, Q1 BSS138, Q16 BSS138, Q3 BSS138, Q4 BSS138, U2 LM2596S-ADJ, U3 LM2596S-ADJ, U4 LM2596S-ADJ, U5 LMV358IDR, U6 LMV358IDR

Commit message: Update Rev-C regulator and HAT designs
Parts:
- removed the C11 at (156.8, 84.2)
- removed the C2 at (158.4, 66.9)
- removed the C3 at (171.0, 90.1)
- removed the C4 at (147.6, 71.8)
- removed the C5 at (158.7, 97.1)
- removed the D1 at (146.6, 80.8)
- removed the D3 at (159.7, 88.9)
- removed L5: 33uh, Inductor_SMD:L_11.5x10mm_H6mm
- removed the R11 at (162.6, 84.2)
- removed the R15 at (219.6, 122.6)
- removed the R25 at (208.3, 147.1)
- removed the R27 at (167.5, 148.9)
- removed the R29 at (162.6, 88.9)
- removed the R3 at (167.3, 66.8)
- removed the U2 at (165.8, 75.1)
- added C13: 100nF, Capacitor_SMD:C_0805_2012Metric, F.Cu at (84.7, 116.9)
- added C16: 100nF, PCM_JLCPCB:C_0805, F.Cu at (93.1, 90.4)
- added C18: 100nF, PCM_JLCPCB:C_0805, F.Cu at (-44.0, 122.3)
- added C19: 100nF, PCM_JLCPCB:C_0805, F.Cu at (93.1, 96.5)
- added C20: 100nF, PCM_JLCPCB:C_0805, F.Cu at (93.1, 99.6)
- added C22: 100nF, PCM_JLCPCB:C_0805, F.Cu at (-39.4, 122.6)
- added C23: 100nF, PCM_JLCPCB:C_0805, F.Cu at (-11.5, 119.2)
- added C24: 100nF, PCM_JLCPCB:C_0805, F.Cu at (-11.5, 116.7)
- added C25: 10uF, PCM_JLCPCB:C_0805, F.Cu at (93.1, 111.8)
- added C26: 10uF, PCM_JLCPCB:C_0805, F.Cu at (-44.8, 112.2)
- added C27: 100nF, PCM_JLCPCB:C_0805, F.Cu at (-37.2, 138.0)
- added C28: 100nF, PCM_JLCPCB:C_0805, F.Cu at (-28.1, 138.3)
- added C29: 100nF, PCM_JLCPCB:C_0805, F.Cu at (46.4, 143.3)
- added C30: 100nF, PCM_JLCPCB:C_0805, F.Cu at (32.8, 143.3)
- added C31: 10uF, PCM_JLCPCB:C_0805, F.Cu at (57.5, 145.5)
- added C32: 10uF, PCM_JLCPCB:C_0805, F.Cu at (-17.8, 147.1)
- added C33: 470uf, Capacitor_SMD:CP_Elec_10x10, F.Cu at (-43.7, 129.2)
- added C34: 470uf, Capacitor_SMD:CP_Elec_10x10, F.Cu at (26.2, 129.8)
- added C35: 1nF, PCM_JLCPCB:C_0805, F.Cu at (85.3, 147.4)
- added C36: 1nF, PCM_JLCPCB:C_0805, F.Cu at (-4.52, 114.3)
- added C37: 1nF, PCM_JLCPCB:C_0805, F.Cu at (84.7, 140.5)
- added C38: 1nF, PCM_JLCPCB:C_0805, F.Cu at (-4.52, 120.8)
- added C39: 100nF, PCM_JLCPCB:C_0805, F.Cu at (84.1, 137.5)
- added C40: 100nF, PCM_JLCPCB:C_0805, F.Cu at (-4.52, 129.1)
- added C41: 100nF, PCM_JLCPCB:C_0805, F.Cu at (63.7, 133.8)
- added C42: 100nF, PCM_JLCPCB:C_0805, F.Cu at (-10.8, 134.2)
- added C43: 100nF, PCM_JLCPCB:C_0805, F.Cu at (102.0, 111.8)
- added C44: 100nF, PCM_JLCPCB:C_0805, F.Cu at (106.4, 90.4)
- added C45: 100nF, PCM_JLCPCB:C_0805, F.Cu at (-45.8, 143.2)
- added C46: 100nF, PCM_JLCPCB:C_0805, F.Cu at (-45.8, 145.6)
- added C47: 100nF, PCM_JLCPCB:C_0805, F.Cu at (-38.0, 152.4)
- added D10: 1SMA4742A, PCM_JLCPCB:D_DO-214AC(SMA), F.Cu at (-22.3, 126.5)
- added D11: 1SMA4742A, PCM_JLCPCB:D_DO-214AC(SMA), F.Cu at (77.6, 104.1)
- added D12: SMBJ6.0CA, PCM_JLCPCB:D_SMB, F.Cu at (-43.5, 139.2)
- added D13: SMBJ6.0CA, PCM_JLCPCB:D_SMB, F.Cu at (25.6, 139.9)
- added D14: Green, PCM_JLCPCB:D_0805, F.Cu at (-21.8, 154.7)
- added D15: Green, PCM_JLCPCB:D_0805, F.Cu at (49.6, 155.1)
- added D16: 1N5819WS, Diode_SMD:D_SOD-323, F.Cu at (130.6, 77.2)
- added D17: 1N5819WS, Diode_SMD:D_SOD-323, F.Cu at (-4.50, 106.3)
- added D8: 1SMA4742A, PCM_JLCPCB:D_DO-214AC(SMA), F.Cu at (-31.4, 126.6)
- added D9: 1SMA4742A, PCM_JLCPCB:D_DO-214AC(SMA), F.Cu at (77.6, 96.0)
- added J10: 1935161, digikey-footprints:Terminal_Block_D1.3mm_P5mm, F.Cu at (36.7, 152.8)
- added J11: 1935161, digikey-footprints:Terminal_Block_D1.3mm_P5mm, F.Cu at (-32.9, 153.5)
- added J8: Conn_01x20_Pin, Connector_PinHeader_2.54mm:PinHeader_1x20_P2.54mm_Horizontal, F.Cu at (-52.5, 144.5)
- added L3: L_Ferrite, Inductor_SMD:L_1206_3216Metric, F.Cu at (-32.6, 146.3)
- added L4: L_Ferrite, Inductor_SMD:L_1206_3216Metric, F.Cu at (35.4, 146.3)
- added POT1: 3296W-1-103LF, Potentiometer_THT:Potentiometer_Bourns_3296W_Vertical, F.Cu at (71.0, 117.9)
- added POT2: 3296W-1-103LF, Potentiometer_THT:Potentiometer_Bourns_3296W_Vertical, F.Cu at (71.0, 129.1)
- added POT3: 3296W-1-103LF, Potentiometer_THT:Potentiometer_Bourns_3296W_Vertical, F.Cu at (0.52, 119.8)
- added POT4: 3296W-1-103LF, Potentiometer_THT:Potentiometer_Bourns_3296W_Vertical, F.Cu at (0.52, 134.2)
- added Q10: PSMN5R2-60YL, Package_TO_SOT_SMD:LFPAK56, F.Cu at (-22.1, 131.1)
- added Q11: PSMN5R2-60YL, Package_TO_SOT_SMD:LFPAK56, F.Cu at (39.5, 131.3)
- added Q12: PSMN5R2-60YL, Package_TO_SOT_SMD:LFPAK56, F.Cu at (52.1, 131.1)
- added Q5: PSMN5R2-60YL, Package_TO_SOT_SMD:LFPAK56, F.Cu at (-31.5, 119.9)
- added Q6: PSMN5R2-60YL, Package_TO_SOT_SMD:LFPAK56, F.Cu at (38.6, 120.4)
- added Q7: PSMN5R2-60YL, Package_TO_SOT_SMD:LFPAK56, F.Cu at (-22.1, 119.4)
- added Q8: PSMN5R2-60YL, Package_TO_SOT_SMD:LFPAK56, F.Cu at (51.9, 120.2)
- added Q9: PSMN5R2-60YL, Package_TO_SOT_SMD:LFPAK56, F.Cu at (-31.7, 131.3)
- added R23: 10Ω, PCM_JLCPCB:R_0805, F.Cu at (93.1, 57.9)
- added R31: 390kΩ, PCM_JLCPCB:R_0805, F.Cu at (93.1, 63.8)
- added R32: 100kΩ, PCM_JLCPCB:R_0805, F.Cu at (-13.9, 150.3)
- added R33: 100kΩ, PCM_JLCPCB:R_0805, F.Cu at (93.1, 69.7)
- added R34: 10Ω, PCM_JLCPCB:R_0805, F.Cu at (-39.3, 121.0)
- added R37: 100kΩ, PCM_JLCPCB:R_0805, F.Cu at (93.1, 75.6)
- added R38: 390kΩ, PCM_JLCPCB:R_0805, F.Cu at (93.1, 78.6)
- added R39: 100kΩ, PCM_JLCPCB:R_0805, F.Cu at (93.1, 81.5)
- added R40: 390kΩ, PCM_JLCPCB:R_0805, F.Cu at (-39.2, 116.3)
- added R42: 100kΩ, PCM_JLCPCB:R_0805, F.Cu at (-39.3, 118.6)
- added R43: 100kΩ, PCM_JLCPCB:R_0805, F.Cu at (97.5, 60.9)
- added R44: 20m ohms, Resistor_SMD:R_2512_6332Metric, F.Cu at (-33.5, 139.3)
- added R45: 20mΩ, Resistor_SMD:R_2512_6332Metric, F.Cu at (37.5, 138.6)
- added R46: 100kΩ, PCM_JLCPCB:R_0805, F.Cu at (-32.0, 123.8)
- added R47: 200mΩ, Resistor_SMD:R_2512_6332Metric, F.Cu at (51.1, 139.7)
- added R48: 10Ω, PCM_JLCPCB:R_0805, F.Cu at (-37.4, 141.8)
- added R49: 10Ω, PCM_JLCPCB:R_0805, F.Cu at (-16.1, 116.8)
- added R50: 10Ω, PCM_JLCPCB:R_0805, F.Cu at (-37.4, 144.7)
- added R51: 10Ω, PCM_JLCPCB:R_0805, F.Cu at (32.8, 138.6)
- added R52: 200m ohms, Resistor_SMD:R_2512_6332Metric, F.Cu at (-23.6, 139.5)
- added R53: 10Ω, PCM_JLCPCB:R_0805, F.Cu at (-28.2, 143.1)
- added R54: 10Ω, PCM_JLCPCB:R_0805, F.Cu at (33.0, 141.0)
- added R55: 390kΩ, PCM_JLCPCB:R_0805, F.Cu at (-16.0, 119.2)
- added R56: 100kΩ, PCM_JLCPCB:R_0805, F.Cu at (-22.5, 123.8)
- added R57: 10Ω, PCM_JLCPCB:R_0805, F.Cu at (46.5, 138.7)
- added R58: 10Ω, PCM_JLCPCB:R_0805, F.Cu at (-28.2, 140.8)
- added R59: 10Ω, PCM_JLCPCB:R_0805, F.Cu at (46.5, 141.0)
- added R60: 270Ω, PCM_JLCPCB:R_0805, F.Cu at (-21.9, 152.0)
- added R61: 100kΩ, PCM_JLCPCB:R_0805, F.Cu at (-16.1, 121.9)
- added R62: 270Ω, PCM_JLCPCB:R_0805, F.Cu at (49.6, 153.0)
- added R63: 10Ω, PCM_JLCPCB:R_0805, F.Cu at (-17.8, 150.2)
- added R64: 10Ω, PCM_JLCPCB:R_0805, F.Cu at (57.5, 147.8)
- added R65: 10Ω, PCM_JLCPCB:R_0805, F.Cu at (-17.9, 152.8)
- added R66: 10Ω, PCM_JLCPCB:R_0805, F.Cu at (-38.1, 154.9)
- added R67: 10Ω, PCM_JLCPCB:R_0805, F.Cu at (57.5, 150.0)
- added R68: 10Ω, PCM_JLCPCB:R_0805, F.Cu at (106.3, 57.9)
- added R69: 10kΩ, PCM_JLCPCB:R_0805, F.Cu at (57.5, 138.8)
- added R70: 10kΩ, PCM_JLCPCB:R_0805, F.Cu at (57.5, 141.0)
- added R71: 10kΩ, PCM_JLCPCB:R_0805, F.Cu at (69.0, 142.6)
- added R72: 10kΩ, PCM_JLCPCB:R_0805, F.Cu at (69.0, 140.1)
- added R73: 10kΩ, PCM_JLCPCB:R_0805, F.Cu at (-18.0, 142.0)
- added R74: 10kΩ, PCM_JLCPCB:R_0805, F.Cu at (-17.8, 139.2)
- added R75: 10kΩ, PCM_JLCPCB:R_0805, F.Cu at (-4.40, 141.5)
- added R76: 10kΩ, PCM_JLCPCB:R_0805, F.Cu at (-4.44, 138.2)
- added R77: 510kΩ, PCM_JLCPCB:R_0805, F.Cu at (57.5, 143.3)
- added R78: 510kΩ, PCM_JLCPCB:R_0805, F.Cu at (91.5, 117.9)
- added R79: 510kΩ, PCM_JLCPCB:R_0805, F.Cu at (-17.9, 144.3)
- added R80: 510kΩ, PCM_JLCPCB:R_0805, F.Cu at (-4.42, 144.8)
- added R81: 510kΩ, PCM_JLCPCB:R_0805, F.Cu at (57.5, 136.6)
- added R82: 510kΩ, PCM_JLCPCB:R_0805, F.Cu at (69.0, 137.2)
- added R83: 510kΩ, PCM_JLCPCB:R_0805, F.Cu at (-17.7, 136.9)
- added R85: 1kΩ, PCM_JLCPCB:R_0805, F.Cu at (59.7, 134.0)
- added R86: 1kΩ, PCM_JLCPCB:R_0805, F.Cu at (84.4, 143.4)
- added R87: 1kΩ, PCM_JLCPCB:R_0805, F.Cu at (-14.8, 134.2)
- added R88: 1kΩ, PCM_JLCPCB:R_0805, F.Cu at (-4.52, 125.2)
- added R89: 10kΩ, PCM_JLCPCB:R_0805, F.Cu at (110.7, 87.4)
- added R90: 10kΩ, PCM_JLCPCB:R_0805, F.Cu at (-4.52, 117.4)
- added R91: 10kΩ, PCM_JLCPCB:R_0805, F.Cu at (68.2, 147.9)
- added R92: 10kΩ, PCM_JLCPCB:R_0805, F.Cu at (-4.52, 132.3)
- added R93: 100kΩ, PCM_JLCPCB:R_0805, F.Cu at (115.1, 66.8)
- added R94: 100kΩ, PCM_JLCPCB:R_0805, F.Cu at (-4.52, 108.6)
- added TP3: TestPoint_Small, Connector_PinHeader_2.54mm:PinHeader_1x01_P2.54mm_Vertical, F.Cu at (0.51, 99.8)
- added TP4: TestPoint_Small, Connector_PinHeader_1.00mm:PinHeader_1x01_P1.00mm_Vertical, F.Cu at (133.1, 90.4)
- added TP5: TestPoint_Small, Connector_PinHeader_1.00mm:PinHeader_1x01_P1.00mm_Vertical, F.Cu at (0.51, 111.2)
- added TP6: TestPoint_Small, Connector_PinHeader_1.00mm:PinHeader_1x01_P1.00mm_Vertical, F.Cu at (133.1, 96.5)
- added TP7: TestPoint_Small, Connector_PinHeader_1.00mm:PinHeader_1x01_P1.00mm_Vertical, F.Cu at (0.51, 124.8)
- added TP8: TestPoint_Small, Connector_PinHeader_1.00mm:PinHeader_1x01_P1.00mm_Vertical, F.Cu at (133.1, 102.6)
- added TP9: TestPoint_Small, Connector_PinHeader_1.00mm:PinHeader_1x01_P1.00mm_Vertical, F.Cu at (0.51, 105.7)
- added U10: INA2180A2IDGKR, Package_SO:VSSOP-8_3x3mm_P0.65mm, F.Cu at (-10.8, 140.2)
- added U11: TLV1702AIDGKR, Package_SO:Texas_S-PDSO-G8_3x3mm_P0.65mm, F.Cu at (62.4, 129.5)
- added U12: TLV1702AIDGKR, Package_SO:Texas_S-PDSO-G8_3x3mm_P0.65mm, F.Cu at (-11.2, 129.5)
- added U13: INA3221, Package_DFN_QFN:Texas_RGV0016A_VQFN-16-1EP_4x4mm_P0.65mm_EP2.1x2.1mm, F.Cu at (22.1, 151.4)
- added U14: INA3221, Package_DFN_QFN:Texas_RGV0016A_VQFN-16-1EP_4x4mm_P0.65mm_EP2.1x2.1mm, F.Cu at (-45.4, 150.1)
- added U3: LM74502DDFR, Package_TO_SOT_SMD:TSOT-23-8, F.Cu at (24.5, 119.5)
- added U6: LM74502DDFR, Package_TO_SOT_SMD:TSOT-23-8, F.Cu at (62.4, 121.8)
- added U7: LM74502DDFR, Package_TO_SOT_SMD:TSOT-23-8, F.Cu at (-43.9, 119.1)
- added U8: LM74502DDFR, Package_TO_SOT_SMD:TSOT-23-8, F.Cu at (-11.5, 122.3)
- added U9: INA2180A2IDGKR, Package_SO:VSSOP-8_3x3mm_P0.65mm, F.Cu at (63.0, 140.4)
- 10mm2: moved to F.Cu
- C1: renamed from C23; footprint PCM_JLCPCB:C_0805 -> Capacitor_SMD:C_0805_2012Metric
- C10: renamed from C21; footprint PCM_JLCPCB:C_0805 -> Capacitor_SMD:C_0805_2012Metric
- C11: renamed from C7; footprint PCM_JLCPCB:C_0805 -> Capacitor_SMD:C_0805_2012Metric
- C14: renamed from C15; footprint PCM_JLCPCB:C_0805 -> Capacitor_SMD:C_0805_2012Metric
- C2: renamed from C17; footprint PCM_JLCPCB:C_0805 -> Capacitor_SMD:C_0805_2012Metric
- C5: renamed from C26; footprint PCM_JLCPCB:C_0805 -> Capacitor_SMD:C_0805_2012Metric
- C6: renamed from C19; footprint PCM_JLCPCB:C_0805 -> Capacitor_SMD:C_0805_2012Metric
- C7: renamed from C16; footprint PCM_JLCPCB:C_0805 -> Capacitor_SMD:C_0805_2012Metric
- L1: footprint Inductor_SMD:L_11.5x10mm_H6mm -> Inductor_SMD:L_Sunlord_MWSA1003S
- L2: renamed from L3; footprint Inductor_SMD:L_11.5x10mm_H6mm -> Inductor_SMD:L_Sunlord_MWSA1003S
- R25: renamed from R14; value 1kΩ -> 820Ω
- R26: renamed from R22; value 2kΩ -> 1.8kΩ
- R29: renamed from R33; value 100Ω -> 1kΩ
- R41: value 3100 -> 100kΩ
- RT1: footprint 1My_Parts_ Passive:Inrush limiter -> Varistor:RV_Disc_D7mm_W4.5mm_P5mm
- U4: renamed from U6; value LMV358IDR -> TLV9352
- U5: value LMV358IDR -> TLV9352
- moved 10mm1 290.1 mm to (-80.4, 88.5), turned to 0 degrees
- moved C3 271.5 mm to (-49.2, 88.7), turned to 180 degrees
- moved C14 261.0 mm to (-48.6, 112.3)
- moved R6 259.5 mm to (-47.8, 96.3), turned to 0 degrees
- moved C7 257.8 mm to (-40.0, 91.3), turned to 90 degrees
- moved U2 255.5 mm to (-33.0, 89.7), turned to 90 degrees
- moved 10mm2 251.5 mm to (-86.1, 104.0), turned to 0 degrees
- moved D4 250.1 mm to (-47.3, 104.3), turned to -90 degrees
- moved R15 247.9 mm to (-24.4, 98.5), turned to 180 degrees
- moved Q3 247.6 mm to (-18.9, 98.5)
- moved Q2 247.3 mm to (-19.0, 93.5)
- moved R27 243.0 mm to (-24.3, 85.6), turned to 0 degrees
- moved R12 242.5 mm to (-13.3, 98.4)
- moved R8 241.9 mm to (-13.2, 92.9)
- moved R25 241.8 mm to (-24.3, 88.9), turned to 0 degrees
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- renumbered C20 to C12, C22 to C15, C9 to C17, C10 to C21, C12 to C3, C18 to C4, C25 to C8, C13 to C9, D7 to D1, D8 to D2, D2 to D3, D9 to D4, D11 to D5, D5 to D6, D4 to D7, H2 to H1, H3 to H2, H1 to H3, J3 to J1, J5 to J2, J4 to J3, J1 to J4, J2 to J5, Q3 to Q1, Q16 to Q2, Q4 to Q3, Q1 to Q4, R39 to R1, R6 to R10, R8 to R11, R40 to R12, R5 to R13, R9 to R14, R1 to R15, R38 to R16, R44 to R17, R10 to R18, R18 to R19, R37 to R2, R7 to R20, R19 to R21, R13 to R22, R20 to R24, R23 to R27, R49 to R3, R34 to R30, R31 to R35, R32 to R36, R48 to R4, R12 to R5, R16 to R6, R24 to R7, R2 to R8, R4 to R9, TP2 to TP1, TP1 to TP2, TP4 to TP3, U4 to U1, U3 to U2
Connections:
- C10 pad 2: Net-(U4-FB) -> Net-(U1-FB)
- C17 pad 1: +5V_Boot -> +12V
- C21 pad 1: +5V_Boot -> +12V
- J4 pad 06: Incoming (+) -> unconnected-(J4-Pad06)
- J4 pad 08: Incoming (-) -> unconnected-(J4-Pad08)
- J4 pad 12: FAULT_CRITICAL_SUM -> unconnected-(J4-Pad12)
- J4 pad 15: ISET_MPU_3V3 -> unconnected-(J4-Pad15)
- J4 pad 17: VSENSE_3V3- -> unconnected-(J4-Pad17)
- J4 pad 19: VSENSE_3V3+ -> unconnected-(J4-Pad19)
- J5 pad 09: +3.3V_Reg -> Net-(J5-Pad09)
- J5 pad 11: +3.3V_Reg -> Net-(J5-Pad09)
- J5 pad 13: +3.3V_Reg -> Net-(J5-Pad09)
- J5 pad 15: +3.3V_Reg -> Net-(J5-Pad09)
- J5 pad 17: +3.3V_Reg -> Net-(J5-Pad09)
- R19 pad 1: Net-(U4-FB) -> Net-(U1-FB)
- R21 pad 1: Net-(U4-FB) -> Net-(U1-FB)
- R28 pad 1: VSENSE_5V- -> Net-(U6-GATE)
- R28 pad 2: Net-(U4-FB) -> Gate _5_LOW
- R41 pad 1: Net-(U2-FB) (its old number) -> SRC 5_HIGH
- R41 pad 2: +5V_Boot -> Gate _5_High
- U1 pad 4: Net-(U4-FB) -> Net-(U1-FB)
- U4 pad 8: +5V_Boot -> +12V
- U5 pad 8: +5V_Boot -> +12V
Routing:
- net +5V_Boot: track 214.6 -> 0.00 mm, vias 9 -> 0
- net GND: track 191.7 -> 0.00 mm, vias 11 -> 0
- net FAULT_CRITICAL_SUM: track 178.4 -> 0.00 mm, vias 4 -> 0
- net +12V: track 125.0 -> 3.21 mm, vias 2 -> 0
- net Net-(Q4-G): track 119.0 -> 0.00 mm, vias 3 -> 0
- net +5V_reg: track 108.5 -> 0.00 mm, vias 3 -> 0
- net VSENSE_5V+: track 104.6 -> 0.00 mm, vias 2 -> 0
- net VSENSE_3V3+: track 72.9 -> 0.00 mm, vias 2 -> 0
- net Net-(C5-Pad1): track 69.3 -> 0.00 mm, vias 2 -> 0
- net VSENSE_5V-: track 66.0 -> 0.00 mm, vias 4 -> 0
- net ISET_MPU_3V3: track 65.1 -> 0.00 mm, vias 4 -> 0
- net Net-(U1-VIN): track 58.8 -> 0.00 mm
- net +3.3V_Reg: track 76.7 -> 19.8 mm, vias 2 -> 0
- net ISET_MPU_5V: track 56.4 -> 0.00 mm, vias 4 -> 0
- net Net-(J2-Pin_1): track 54.4 -> 0.00 mm
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Other:
- board size 100 x 100 mm -> 291.9 x 100.9 mm
- board text removed: "+5v Boot"
