File: hardware/kicad/dsp-regulator-rev-c/DSP-Regulator-RevC.kicad_sch (KiCad schematic)
At the start: 97 parts, among them J1 CLP-110-02-X-D, J2 CLP-110-02-X-D, J3 1935161, J4 Wire con, J5 Wire con, Q1 BSS138, Q16 BSS138, Q3 BSS138, Q4 BSS138, U2 LM2596S-ADJ, U3 LM2596S-ADJ, U4 LM2596S-ADJ, U5 LMV358IDR, U6 LMV358IDR

Commit message: Sync regulator Rev-C design baseline
Parts:
- removed R15, R25, R27, R28: 10Ω, PCM_JLCPCB:R_0805, symbol PCM_JLCPCB-Resistors:0805,10Ω
- removed unit 2 of U5
- added R32, R33: 100kΩ, PCM_JLCPCB:R_0805, symbol PCM_JLCPCB-Resistors:0805,100kΩ
- added unit 2 of U5
- R25: renamed from R14; value 1kΩ -> 820Ω; symbol PCM_JLCPCB-Resistors:0805,1kΩ -> PCM_JLCPCB-Resistors:0805,820Ω; Class Basic Component -> Preferred Component; LCSC C17513 -> C17837; Part 0805W8F1001T5E -> 0805W8F8200T5E; Resistance 1kΩ -> 820Ω; Stock 7431283 -> 155965
- R26: renamed from R22; value 2kΩ -> 1.8kΩ; symbol PCM_JLCPCB-Resistors:0805,2kΩ -> PCM_JLCPCB-Resistors:0805,1.8kΩ; Class Basic Component -> Preferred Component; LCSC C17604 -> C17398; Part 0805W8F2001T5E -> 0805W8F1801T5E; Resistance 2kΩ -> 1.8kΩ; Stock 2296950 -> 170330
- R29: renamed from R33; value 100Ω -> 1kΩ; symbol PCM_JLCPCB-Resistors:0805,100Ω -> PCM_JLCPCB-Resistors:0805,1kΩ; LCSC C17408 -> C17513; Part 0805W8F1000T5E -> 0805W8F1001T5E; Resistance 100Ω -> 1kΩ; Stock 3356429 -> 7431283
- U4: renamed from U6; value LMV358IDR -> TLV9352; symbol dk_Linear-Amplifiers-Instrumentation-OP-Amps-Buffer-Amps:LMV358IDR -> 1My_IC's:TLV9352; LCSC (none) -> C4366962
- U5: value LMV358IDR -> TLV9352; symbol dk_Linear-Amplifiers-Instrumentation-OP-Amps-Buffer-Amps:LMV358IDR -> 1My_IC's:TLV9352; LCSC (none) -> C4366962
- renumbered 10mm2 to 10mm1, 10mm1 to 10mm2, C23 to C1, C21 to C10, C7 to C11, C20 to C12, C4 to C13, C15 to C14, C22 to C15, C2 to C16, C9 to C17, C11 to C18, C3 to C19, C17 to C2, C5 to C20, C10 to C21, C12 to C3, C18 to C4, C26 to C5, C19 to C6, C16 to C7, C25 to C8, C13 to C9, D7 to D1, D8 to D2, D2 to D3, D9 to D4, D11 to D5, D5 to D6, D4 to D7, D1 to D8, D3 to D9, H2 to H1, H3 to H2, H1 to H3, J3 to J1, J5 to J2, J4 to J3, J1 to J4, J2 to J5, L3 to L2, L5 to L3, Q3 to Q1, Q16 to Q2, Q4 to Q3, Q1 to Q4, R39 to R1, R6 to R10, R8 to R11, R40 to R12, R5 to R13, R9 to R14, R1 to R15, R38 to R16, R44 to R17, R10 to R18, R18 to R19, R37 to R2, R7 to R20, R19 to R21, R13 to R22, R3 to R23, R20 to R24, R23 to R27, R11 to R28, R49 to R3, R34 to R30, R41 to R31, R29 to R34, R31 to R35, R32 to R36, R48 to R4, R12 to R5, R16 to R6, R24 to R7, R2 to R8, R4 to R9, TP2 to TP1, TP1 to TP2, TP4 to TP3, U4 to U1, U3 to U2, U2 to U3
Connections:
- net +12V: now also C17.1, C21.1, U4.8 (VCC+), U4.8 (VCC+), U5.8 (VCC+)
- net +5V_Boot: no longer C17.1, C21.1, U4.8 (VCC+)
- net GND: now also U4.4 (GND), R32.2, R33.2, U5.4 (GND)
- net VSENSE_3V3+: now also R32.1
- net VSENSE_5V+: now also R33.1
- net at R35.2, R36.1: now also U5.5
- net at D7.2 (A): now also U5.6, U5.7
Other:
- moved on the sheet: C17, R35, R36

Commit message: Update Rev-C regulator and HAT designs
Parts:
- removed C13: 470uf 25V, Capacitor_SMD:CP_Elec_10x10.5, symbol Device:C_Polarized_US
- removed C16, C20: 100nF, PCM_JLCPCB:C_0805, symbol PCM_JLCPCB-Capacitors:0805,100nF
- removed C18: 100pF, PCM_JLCPCB:C_0805, symbol PCM_JLCPCB-Capacitors:0805,100pF
- removed C19: 330uF 25v, Capacitor_SMD:CP_Elec_10x10.5, symbol Device:C_Polarized_US
- removed D8: SS54B, PCM_JLCPCB:D_SMB, symbol PCM_JLCPCB-Diodes:Schottky,SS54B
- removed D9: Yellow, PCM_JLCPCB:D_0805, symbol PCM_JLCPCB-Diodes_1:LED,0805,Yellow
- removed J4, J5: CLP-110-02-X-D, 1My_Parts_ Connectors:SAMTEC_CLP-110-02-X-D, symbol 1My_Connectors:CLP-110-02-X-D
- removed L3: 33uh, Inductor_SMD:L_11.5x10mm_H6mm, symbol Device:L
- removed R23: 0Ω, PCM_JLCPCB:R_1206, symbol PCM_JLCPCB-Resistors:1206,0Ω
- removed R28: 1k, PCM_JLCPCB:R_0805, symbol PCM_JLCPCB-Resistors:0805,1kΩ
- removed R31: 3100, PCM_JLCPCB:R_0805, symbol PCM_JLCPCB-Resistors:0805,100Ω
- removed R34: 680Ω, PCM_JLCPCB:R_0805, symbol PCM_JLCPCB-Resistors:0805,680Ω
- removed U3: LM2596S-ADJ, Package_TO_SOT_SMD:TO-263-5_TabPin3, symbol Regulator_Switching:LM2596S-ADJ
- added C13: 100nF, Capacitor_SMD:C_0805_2012Metric, symbol PCM_JLCPCB-Capacitors:0805,100nF,(2)
- added C16, C18, C19, C20, C22, C23, C24, C27, C28, C29, C30, C39, C40, C41, C42, C43, C44, C45, C46, C47: 100nF, PCM_JLCPCB:C_0805, symbol PCM_JLCPCB-Capacitors:0805,100nF,(2)
- added C25, C26, C31, C32: 10uF, PCM_JLCPCB:C_0805, symbol PCM_JLCPCB-Capacitors:0805,10uF,(2)
- added C33, C34: 470uf, Capacitor_SMD:CP_Elec_10x10, symbol Device:C_Small_US
- added C35, C36, C37, C38: 1nF, PCM_JLCPCB:C_0805, symbol PCM_JLCPCB-Capacitors:0805,1nF
- added D10, D11, D8, D9: 1SMA4742A, PCM_JLCPCB:D_DO-214AC(SMA), symbol PCM_JLCPCB-Diodes:Zener,1SMA4742A
- added D12, D13: SMBJ6.0CA, PCM_JLCPCB:D_SMB, symbol PCM_JLCPCB-Diodes:TVS-Bi,SMBJ6.0CA
- added D14, D15: Green, PCM_JLCPCB:D_0805, symbol PCM_JLCPCB-Diodes:LED,0805,Green
- added D16, D17: 1N5819WS, Diode_SMD:D_SOD-323, symbol Diode:1N5819WS
- added J10, J11: 1935161, digikey-footprints:Terminal_Block_D1.3mm_P5mm, symbol dk_Terminal-Blocks-Wire-to-Board:1935161
- added J8, J9: Conn_01x20_Pin, Connector_PinHeader_2.54mm:PinHeader_1x20_P2.54mm_Horizontal, symbol Connector:Conn_01x20_Pin
- added L3, L4: L_Ferrite, Inductor_SMD:L_1206_3216Metric, symbol Device:L_Ferrite
- added POT1, POT2, POT3, POT4: 3296W-1-103LF, Potentiometer_THT:Potentiometer_Bourns_3296W_Vertical, symbol 1My_Basic components:3296W-1-103LF
- added Q10, Q11, Q12, Q5, Q6, Q7, Q8, Q9: PSMN5R2-60YL, Package_TO_SOT_SMD:LFPAK56, symbol Transistor_FET:PSMN5R2-60YL
- added R23, R28, R34, R48, R49, R50, R51, R53, R54, R57, R58, R59, R63, R64, R65, R66, R67, R68: 10Ω, PCM_JLCPCB:R_0805, symbol PCM_JLCPCB-Resistors:0805,10Ω
- added R31, R38, R40, R55: 390kΩ, PCM_JLCPCB:R_0805, symbol PCM_JLCPCB-Resistors:0805,390kΩ
- added R37, R39, R41, R42, R43, R46, R56, R61, R93, R94: 100kΩ, PCM_JLCPCB:R_0805, symbol PCM_JLCPCB-Resistors:0805,100kΩ
- added R44: 20m ohms, Resistor_SMD:R_2512_6332Metric, symbol Device:R
- added R45: 20mΩ, Resistor_SMD:R_2512_6332Metric, symbol Device:R
- added R47: 200mΩ, Resistor_SMD:R_2512_6332Metric, symbol Device:R
- added R52: 200m ohms, Resistor_SMD:R_2512_6332Metric, symbol Device:R
- added R60, R62: 270Ω, PCM_JLCPCB:R_0805, symbol PCM_JLCPCB-Resistors:0805,270Ω
- added R69, R70, R71, R72, R73, R74, R75, R76, R89, R90, R91, R92: 10kΩ, PCM_JLCPCB:R_0805, symbol PCM_JLCPCB-Resistors:0805,10kΩ
- added R77, R78, R79, R80, R81, R82, R83, R84: 510kΩ, PCM_JLCPCB:R_0805, symbol PCM_JLCPCB-Resistors:0805,510kΩ
- added R85, R86, R87, R88: 1kΩ, PCM_JLCPCB:R_0805, symbol PCM_JLCPCB-Resistors:0805,1kΩ
- added TP4, TP5, TP6, TP7, TP8, TP9: TestPoint_Small, Connector_PinHeader_1.00mm:PinHeader_1x01_P1.00mm_Vertical, symbol Connector:TestPoint_Small
- added U10, U9: INA2180A2IDGKR, Package_SO:VSSOP-8_3x3mm_P0.65mm, symbol Amplifier_Current:INA2180AxxDGK
- added U11, U12: TLV1702AIDGKR, Package_SO:Texas_S-PDSO-G8_3x3mm_P0.65mm, symbol 1My_IC's:TLV1702AIDGKR
- added U13, U14: INA3221, Package_DFN_QFN:Texas_RGV0016A_VQFN-16-1EP_4x4mm_P0.65mm_EP2.1x2.1mm, symbol Power_Management:INA3221
- added U3, U6, U7, U8: LM74502DDFR, Package_TO_SOT_SMD:TSOT-23-8, symbol 1My_IC's:LM74502HDDFR
- C1, C10, C11, C14, C2, C5, C6, C7: footprint PCM_JLCPCB:C_0805 -> Capacitor_SMD:C_0805_2012Metric
- L1, L2: footprint Inductor_SMD:L_11.5x10mm_H6mm -> Inductor_SMD:L_Sunlord_MWSA1003S
- RT1: footprint 1My_Parts_ Passive:Inrush limiter -> Varistor:RV_Disc_D7mm_W4.5mm_P5mm
Connections:
- net +12V: now also C39.1, C40.1, J8.20 (Pin_20), J9.20 (Pin_20), U11.8 (V+), U12.8 (V+)
- net +3.3V_Reg: now also C26.1, Q5.5 (D), Q7.5 (D)
- net +5V_Boot: now also C13.1, C16.1, C18.1, C19.2, C20.2, C22.2, C23.1, C24.2, J8.3 (Pin_3), J9.3 (Pin_3), POT1.1, POT2.1, POT3.1, POT4.1, R31.1, R38.1, R40.1, R55.1, U3.5 (VS), U6.5 (VS), U7.5 (VS), U8.5 (VS)
- net +5V_reg: now also C25.1, Q6.5 (D), Q8.5 (D)
- net FAULT_CRITICAL_SUM: now also D16.1 (K), D17.1 (K), J8.7 (Pin_7), J9.7 (Pin_7), U13.9 (CRITICAL), U14.9 (CRITICAL)
- net GND: now also C19.1, C20.1, C22.1, C24.1, C25.2, C26.2, C31.2, C32.2, C33.2, C34.2, C39.2, C40.2, C41.2, C42.2, C43.2, C44.2, C46.2, C47.2, D12.1, D13.1, J10.1, J11.1, J8.1 (Pin_1), J8.2 (Pin_2), J8.5 (Pin_5), J9.1 (Pin_1), J9.2 (Pin_2), J9.5 (Pin_5), POT1.3, POT2.3, POT3.3, POT4.3, R37.2, R39.2, R42.2, R60.2, R61.2, R62.2, R66.1, R68.1, R77.1, R78.1, R79.1, R80.1, U10.4 (GND), U11.4 (V-), U12.4 (V-), U13.3 (GND), U13.5 (A0), U14.3 (GND), U3.2 (GND), U6.2 (GND), U7.2 (GND), U8.2 (GND), U9.4 (GND)
- net ISET_MPU_3V3: now also J8.10 (Pin_10)
- net ISET_MPU_5V: now also J9.10 (Pin_10)
- net Incoming (+): now also C45.1, J8.14 (Pin_14), U14.2 (IN+3)
- net Incoming (-): now also C45.2, J8.15 (Pin_15), U14.1 (IN-3)
- net VSENSE_3V3+: now also R63.2, R65.2
- net VSENSE_3V3-: now also R66.2
- net VSENSE_5V+: now also R64.2, R67.2
- net VSENSE_5V-: now also R68.2
- new net: R71.2, R78.2, U9.5 (+)
- new net: R72.2, R82.1, U9.6 (-)
- new net: R82.2, R86.1, U9.7
- new net: R73.2, R79.2, U10.3 (+)
- new net: D16.2 (A), R93.2, TP8.1, U11.1 (OUT), U11.7 (OUT)
- new net: C27.1, Q9.5 (D), R44.1, R48.1
- new net: C27.2, C28.1, C32.1, C33.1, D12.2, L3.1, R44.2, R50.1, R52.2, R53.1, R63.1
- new net: POT4.2, R92.1
- new net: C18.2, U7.4 (VCAP)
- new net: R34.1, U7.6 (GATE)
- new net: R40.2, R42.1, U7.7 (OV)
- new net: C36.2, R87.1, TP5.1, U12.3 (IN+)
- new net: C37.2, R86.2, TP6.1, U11.5 (IN+)
- new net: D15.1, R62.1
- new net: R83.2, R87.2, U10.1
- new net: R74.2, R83.1, U10.2 (-)
- new net: R28.1, U6.6 (GATE)
- new net: C38.1, R92.2, U12.6 (IN-)
- new net: C37.1, R91.2, U11.6 (IN-)
- new net: C47.1, U14.13 (TC)
- new net: C28.2, Q10.5 (D), R52.1, R58.1
- new net: C23.2, U8.4 (VCAP)
- new net: C36.1, R90.2, U12.2 (IN-)
- new net: D14.1, R60.1
- new net: R81.2, R85.2, U9.1
- new net: R70.2, R81.1, U9.2 (-)
- new net: R69.2, R77.2, U9.3 (+)
- new net: C29.2, Q12.5 (D), R47.1, R59.1
- new net: R75.2, R80.2, U10.5 (+)
- new net: D17.2 (A), R94.2, TP9.1, U12.1 (OUT), U12.7 (OUT)
- new net: POT2.2, R91.1
- new net: C35.2, R85.1, TP4.1, U11.3 (IN+)
- new net: POT1.2, R89.1
- new net: POT3.2, R90.1
- new net: C44.1, U13.13 (TC)
- new net: R55.2, R61.1, U8.7 (OV)
- new net: C35.1, R89.2, U11.2 (IN-)
- new net: R38.2, R39.1, U6.7 (OV)
- new net: C16.2, U6.4 (VCAP)
- new net: C13.2, U3.4 (VCAP)
- new net: R76.2, R84.1, U10.6 (-)
- new net: R84.2, R88.1, U10.7
- new net: C38.2, R88.2, TP7.1, U12.5 (IN+)
- new net: C30.1, Q11.5 (D), R45.1, R51.1
- new net: R49.1, U8.6 (GATE)
- new net: R23.1, U3.6 (GATE)
- new net: R31.2, R37.1, U3.7 (OV)
- new net +3.3V Boot: C41.1, C42.1, C43.1, C46.1, J8.4 (Pin_4), J9.4 (Pin_4), R93.1, R94.1, U10.8 (VS), U13.16 (VPU), U13.4 (VS), U14.16 (VPU), U14.4 (VS), U14.5 (A0), U9.8 (VS)
- new net +3v3V_Hi_Range : R48.2, R73.1, U14.12 (IN+1)
- new net +3v3V_low_Range: R58.2, R75.1, U14.15 (IN+2)
- new net +5V_Hi_Range : R51.2, R69.1, U13.12 (IN+1)
- new net +5V_low_Range: R59.2, R71.1, U13.15 (IN+2)
- new net -3v3V_Hi_Range: R50.2, R74.1, U14.11 (IN-1)
- new net -3v3V_low_Range: R53.2, R76.1, U14.14 (IN-2)
- new net -5V_Hi_Range: R54.2, R70.1, U13.11 (IN-1)
- new net -5V_low_Range: R57.2, R72.1, U13.14 (IN-2)
- new net ESP- GPIO 3.3V High: J8.12 (Pin_12), U7.1 (EN_UVLO)
- new net ESP- GPIO 3.3V Low: J8.11 (Pin_11), U8.1 (EN_UVLO)
- new net ESP- GPIO 5V Hi: J9.12 (Pin_12), U3.1 (EN_UVLO)
- new net ESP- GPIO 5V Low: J9.11 (Pin_11), U6.1 (EN_UVLO)
- new net FAULT_WARNING_SUM: J8.6 (Pin_6), J9.6 (Pin_6), U13.8 (WARNING), U14.8 (WARNING)
- new net Gate _3.3_HIGH: D8.2 (cathode), Q5.4 (G), Q9.4 (G), R34.2, R46.2
- new net Gate _3.3_LOW: D10.2 (cathode), Q10.4 (G), Q7.4 (G), R49.2, R56.2
- new net Gate _5_High: D9.2 (cathode), Q11.4 (G), Q6.4 (G), R23.2, R41.2
- new net Gate _5_LOW: D11.2 (cathode), Q12.4 (G), Q8.4 (G), R28.2, R43.2
- new net I²C SCL_0: J8.9 (Pin_9), J9.9 (Pin_9), U13.6 (SCL), U14.6 (SCL)
- new net I²C SDA_0: J8.8 (Pin_8), J9.8 (Pin_8), U13.7 (SDA), U14.7 (SDA)
- new net SRC 3.3_HIGH: D8.1 (anode), Q5.1 (S), Q5.2 (S), Q5.3 (S), Q9.1 (S), Q9.2 (S), Q9.3 (S), R46.1, U7.8 (SRC)
- new net SRC 3.3_LOW: D10.1 (anode), Q10.1 (S), Q10.2 (S), Q10.3 (S), Q7.1 (S), Q7.2 (S), Q7.3 (S), R56.1, U8.8 (SRC)
- new net SRC 5_HIGH: D9.1 (anode), Q11.1 (S), Q11.2 (S), Q11.3 (S), Q6.1 (S), Q6.2 (S), Q6.3 (S), R41.1, U3.8 (SRC)
- new net SRC 5_LOW: D11.1 (anode), Q12.1 (S), Q12.2 (S), Q12.3 (S), Q8.1 (S), Q8.2 (S), Q8.3 (S), R43.1, U6.8 (SRC)
- new net Shunt -: C29.1, C30.2, C31.1, C34.1, D13.2, L4.1, R45.2, R47.2, R54.1, R57.1, R64.1
- new net V_out +3V3: D14.2, J11.2, L3.2, R65.1
- new net V_out +5V: D15.2, J10.2, L4.2, R67.1
- no-connect marks 3 -> 10
Other:
- note added: "Channel 1 5 volts"
- note added: "Channel 2 3.3 volts"
- note added: "Voltage Measuring"
- note removed: "3100 = 5.04V"
- note removed: "Control Voltage Converter"

Commit message: Update Rev-C coplanar board designs
Parts:
- removed C13: 100nF, Capacitor_SMD:C_0805_2012Metric, symbol PCM_JLCPCB-Capacitors:0805,100nF,(2)
- removed C17, C21: 100nF, PCM_JLCPCB:C_0805, symbol PCM_JLCPCB-Capacitors:0805,100nF
- removed C18, C19, C20, C22, C23, C27, C28, C29, C30: 100nF, PCM_JLCPCB:C_0805, symbol PCM_JLCPCB-Capacitors:0805,100nF,(2)
- removed C25, C26, C31, C32: 10uF, PCM_JLCPCB:C_0805, symbol PCM_JLCPCB-Capacitors:0805,10uF,(2)
- removed C33, C34: 470uf, Capacitor_SMD:CP_Elec_10x10, symbol Device:C_Small_US
- removed D10, D11, D8: 1SMA4742A, PCM_JLCPCB:D_DO-214AC(SMA), symbol PCM_JLCPCB-Diodes:Zener,1SMA4742A
- removed D12, D13: SMBJ6.0CA, PCM_JLCPCB:D_SMB, symbol PCM_JLCPCB-Diodes:TVS-Bi,SMBJ6.0CA
- removed D14, D15: Green, PCM_JLCPCB:D_0805, symbol PCM_JLCPCB-Diodes:LED,0805,Green
- removed D6, D7: BAT54C,215, PCM_JLCPCB:SOT-23-3_L2.9-W1.6-P1.90-LS2.8-BR, symbol PCM_JLCPCB-Diode-Packages:Schottky, BAT54C,215
- removed J10, J11: 1935161, digikey-footprints:Terminal_Block_D1.3mm_P5mm, symbol dk_Terminal-Blocks-Wire-to-Board:1935161
- removed J8, J9: Conn_01x20_Pin, Connector_PinHeader_2.54mm:PinHeader_1x20_P2.54mm_Horizontal, symbol Connector:Conn_01x20_Pin
- removed L3: L_Ferrite, Inductor_SMD:L_1206_3216Metric, symbol Device:L_Ferrite
- removed Q12, Q6, Q9: PSMN5R2-60YL, Package_TO_SOT_SMD:LFPAK56, symbol Transistor_FET:PSMN5R2-60YL
- removed R28, R48, R49, R50, R53, R54, R57, R58, R59, R63, R64, R65, R66, R67, R68: 10Ω, PCM_JLCPCB:R_0805, symbol PCM_JLCPCB-Resistors:0805,10Ω
- removed R29: 1kΩ, PCM_JLCPCB:R_0805, symbol PCM_JLCPCB-Resistors:0805,1kΩ
- removed R30, R36: 33kΩ, PCM_JLCPCB:R_0805, symbol PCM_JLCPCB-Resistors:0805,33kΩ
- removed R31, R38, R40, R55: 390kΩ, PCM_JLCPCB:R_0805, symbol PCM_JLCPCB-Resistors:0805,390kΩ
- removed R32, R33, R37, R39, R41, R42, R43, R46, R56, R61: 100kΩ, PCM_JLCPCB:R_0805, symbol PCM_JLCPCB-Resistors:0805,100kΩ
- removed R35: 100Ω, PCM_JLCPCB:R_0805, symbol PCM_JLCPCB-Resistors:0805,100Ω
- removed R44: 20m ohms, Resistor_SMD:R_2512_6332Metric, symbol Device:R
- removed R47: 200mΩ, Resistor_SMD:R_2512_6332Metric, symbol Device:R
- removed R52: 200m ohms, Resistor_SMD:R_2512_6332Metric, symbol Device:R
- removed R60, R62: 270Ω, PCM_JLCPCB:R_0805, symbol PCM_JLCPCB-Resistors:0805,270Ω
- removed TP3: TestPoint_Small, Connector_PinHeader_2.54mm:PinHeader_1x01_P2.54mm_Vertical, symbol Connector:TestPoint_Small
- removed U3, U6, U7, U8: LM74502DDFR, Package_TO_SOT_SMD:TSOT-23-8, symbol 1My_IC's:LM74502HDDFR
- removed U4, U5: TLV9352, digikey-footprints:SOIC-8_W3.9mm, symbol 1My_IC's:TLV9352
- added C1, C12, C15, C31, C33: 100nF, PCM_JLCPCB:C_0805, symbol PCM_JLCPCB-Capacitors:0805,100nF
- added C10, C21, C23, C7: 10uF, PCM_JLCPCB:C_0805, symbol PCM_JLCPCB-Capacitors:0805,10uF,(2)
- added C11, C3, C36, C41, C45, C49, C51, C52, C53: 100nF, PCM_JLCPCB:C_0805, symbol PCM_JLCPCB-Capacitors:0805,100nF,(2)
- added C22, C6: 470uf, Capacitor_SMD:CP_Elec_10x10, symbol Device:C_Small_US
- added C26: 100pF, PCM_JLCPCB:C_0805, symbol PCM_JLCPCB-Capacitors:0805,100pF
- added C30: 470uf 25V, Capacitor_SMD:CP_Elec_10x10.5, symbol Device:C_Polarized_US
- added C32: 330uF 25v, Capacitor_SMD:CP_Elec_10x10.5, symbol Device:C_Polarized_US
- added C38: 100nF, Capacitor_SMD:C_0805_2012Metric, symbol PCM_JLCPCB-Capacitors:0805,100nF,(2)
- added D1, D8: BAT54C,215, PCM_JLCPCB:SOT-23-3_L2.9-W1.6-P1.90-LS2.8-BR, symbol PCM_JLCPCB-Diode-Packages:Schottky, BAT54C,215
- added D11, D3: SMBJ6.0CA, PCM_JLCPCB:D_SMB, symbol PCM_JLCPCB-Diodes:TVS-Bi,SMBJ6.0CA
- added D12, D4: Green, PCM_JLCPCB:D_0805, symbol PCM_JLCPCB-Diodes:LED,0805,Green
- added D13, D2, D6: 1SMA4742A, PCM_JLCPCB:D_DO-214AC(SMA), symbol PCM_JLCPCB-Diodes:Zener,1SMA4742A
- added D15: Yellow, PCM_JLCPCB:D_0805, symbol PCM_JLCPCB-Diodes:LED,0805,Yellow
- added D18: SS54B, PCM_JLCPCB:D_SMB, symbol PCM_JLCPCB-Diodes:Schottky,SS54B
- added D19: Yellow, PCM_JLCPCB:D_0805, symbol PCM_JLCPCB-Diodes_1:LED,0805,Yellow
- added J1, J2: 1935161, digikey-footprints:Terminal_Block_D1.3mm_P5mm, symbol dk_Terminal-Blocks-Wire-to-Board:1935161
- added J6: Conn_01x03_Pin, Connector_PinHeader_2.54mm:PinHeader_1x03_P2.54mm_Vertical_SMD_Pin1Right, symbol Connector:Conn_01x03_Pin
- added J7: Conn_01x06_Pin, Connector_PinHeader_2.54mm:PinHeader_1x06_P2.54mm_Vertical_SMD_Pin1Right, symbol Connector:Conn_01x06_Pin
- added L1: L_Ferrite, Inductor_SMD:L_1206_3216Metric, symbol Device:L_Ferrite
- added L5: 33uh, Inductor_SMD:L_Sunlord_MWSA1003S, symbol Device:L
- added Q1, Q2, Q4: PSMN5R2-60YL, Package_TO_SOT_SMD:LFPAK56, symbol Transistor_FET:PSMN5R2-60YL
- added R10: 100Ω, PCM_JLCPCB:R_0805, symbol PCM_JLCPCB-Resistors:0805,100Ω
- added R100, R22, R27, R36, R49, R6, R78, R88, R9, R97: 100kΩ, PCM_JLCPCB:R_0805, symbol PCM_JLCPCB-Resistors:0805,100kΩ
- added R12, R15, R17, R20, R38, R4, R40, R41, R46, R75, R8, R82, R92, R98: 10Ω, PCM_JLCPCB:R_0805, symbol PCM_JLCPCB-Resistors:0805,10Ω
- added R13, R29: 33kΩ, PCM_JLCPCB:R_0805, symbol PCM_JLCPCB-Resistors:0805,33kΩ
- added R16, R47, R54: 270Ω, PCM_JLCPCB:R_0805, symbol PCM_JLCPCB-Resistors:0805,270Ω
- added R19: 200mΩ, Resistor_SMD:R_2512_6332Metric, symbol Device:R
- added R28: 1kΩ, PCM_JLCPCB:R_0805, symbol PCM_JLCPCB-Resistors:0805,1kΩ
- added R37: 20m ohms, Resistor_SMD:R_2512_6332Metric, symbol Device:R
- added R42, R43: 10kΩ, PCM_JLCPCB:R_0805, symbol PCM_JLCPCB-Resistors:0805,10kΩ
- added R61: 3100, PCM_JLCPCB:R_0805, symbol PCM_JLCPCB-Resistors:0805,100Ω
- added R65: 1k, PCM_JLCPCB:R_0805, symbol PCM_JLCPCB-Resistors:0805,1kΩ
- added R68: 0Ω, PCM_JLCPCB:R_1206, symbol PCM_JLCPCB-Resistors:1206,0Ω
- added R69: 680Ω, PCM_JLCPCB:R_0805, symbol PCM_JLCPCB-Resistors:0805,680Ω
- added R7: 20mΩ, Resistor_SMD:R_2512_6332Metric, symbol Device:R
- added R77, R85, R96, R99: 390kΩ, PCM_JLCPCB:R_0805, symbol PCM_JLCPCB-Resistors:0805,390kΩ
- added TP2: TestPoint_Small, Connector_PinHeader_2.54mm:PinHeader_1x01_P2.54mm_Vertical, symbol Connector:TestPoint_Small
- added U1, U3: TLV9352, digikey-footprints:SOIC-8_W3.9mm, symbol 1My_IC's:TLV9352
- added U14, U15, U16, U9: LM74502DDFR, Package_TO_SOT_SMD:TSOT-23-8, symbol 1My_IC's:LM74502HDDFR
- added U5: AW9523B, Package_DFN_QFN:QFN-24-1EP_4x4mm_P0.5mm_EP2.7x2.7mm, symbol Interface_Expansion:AW9523B
- added U8: LM2596S-ADJ, Package_TO_SOT_SMD:TO-263-5_TabPin3, symbol Regulator_Switching:LM2596S-ADJ
- Q10: Manufacturer_Name (none) -> Infineon; Manufacturer_Part_Number (none) -> IRLZ44NPBF; Part (none) -> HL3400
- Q11: Manufacturer_Name Infineon -> (none); Manufacturer_Part_Number IRLZ44NPBF -> (none); Part HL3400 -> (none)
- R45: value 20mΩ -> 200m ohms; LCSC C49164694 -> C7420022
- renumbered C1 to C13, C11 to C14, C3 to C17, C7 to C18, C9 to C19, C10 to C2, C14 to C20, C2 to C25, C36 to C27, C5 to C28, C8 to C29, C40 to C34, C42 to C35, C38 to C37, C43 to C39, C46 to C40, C35 to C42, C44 to C43, C47 to C44, C45 to C46, C39 to C47, C41 to C48, C6 to C5, C37 to C50, C12 to C8, C15 to C9, D4 to D10, D2 to D14, D3 to D16, D16 to D20, D1 to D7, H3 to H2, H2 to H3, J2 to J3, J1 to J4, J3 to J5, L1 to L3, POT3 to POT1, POT4 to POT2, POT1 to POT3, POT2 to POT4, Q3 to Q12, Q1 to Q3, Q4 to Q6, Q2 to Q9, R21 to R1, R5 to R11, R13 to R14, R7 to R18, R24 to R2, R9 to R21, R3 to R24, R2 to R25, R16 to R26, R26 to R3, R22 to R30, R25 to R31, R27 to R32, R20 to R33, R6 to R35, R15 to R39, R8 to R44, R10 to R48, R19 to R5, R4 to R50, R1 to R52, R12 to R53, R94 to R55, R87 to R56, R11 to R57, R73 to R58, R14 to R59, R18 to R60, R74 to R62, R90 to R63, R17 to R64, R79 to R66, R83 to R67, R75 to R70, R92 to R71, R76 to R72, R80 to R73, R84 to R74, R88 to R76, R93 to R79, R85 to R80, R69 to R81, R70 to R83, R89 to R84, R77 to R86, R81 to R87, R71 to R89, R91 to R90, R72 to R91, R78 to R93, R82 to R94, R86 to R95, TP2 to TP1, TP1 to TP3, TP5 to TP4, TP9 to TP5, TP7 to TP6, TP4 to TP7, TP6 to TP9, U13 to U10, U14 to U11, U9 to U12, U11 to U13, U1 to U2, U2 to U4, U10 to U6, U12 to U7
Connections:
- net Shunt - is gone; now on an unnamed net: L4.1, R45.2
- net +12V: now also C1.1, C12.1, J7.4 (Pin_4), R68.1, U1.8 (VCC+), U1.8 (VCC+), U3.8 (VCC+), U3.8 (VCC+)
- net +3.3V Boot: now also C15.1, J7.3 (Pin_3), R42.2, R43.2, U5.21 (VCC)
- net +3.3V_Reg: now also Q10.5 (D), C21.1, R28.1; no longer Q5.5 (D)
- net +3v3V_Hi_Range : now also R34.2
- net +3v3V_low_Range: now also R51.2
- net +5V_Boot: now also C26.1, C32.1, C33.1, C36.2, C38.1, C41.2, C45.1, C49.2, C51.1, C52.2, C53.1, D19.2, J7.2 (Pin_2), L5.2, R61.2, R77.1, R85.1, R96.1, R99.1, U14.5 (VS), U15.5 (VS), U16.5 (VS), U9.5 (VS); no longer C16.1, C24.2
- net +5V_Hi_Range : now also R4.2; no longer R51.2
- net +5V_low_Range: now also R23.2
- net +5V_reg: now also C10.1, Q1.5 (D), Q4.5 (D), R10.1; no longer Q8.5 (D)
- net -3v3V_Hi_Range: now also R38.2
- net -3v3V_low_Range: now also R46.2
- net -5V_Hi_Range: now also R8.2
- net -5V_low_Range: now also R20.2
- net ESP- GPIO 3.3V High: now also U15.1 (EN_UVLO), U5.8 (P0_3)
- net ESP- GPIO 3.3V Low: now also U16.1 (EN_UVLO), U5.10 (P0_4)
- net ESP- GPIO 5V Hi: now also U5.6 (P0_1), U9.1 (EN_UVLO)
- net ESP- GPIO 5V Low: now also U14.1 (EN_UVLO), U5.7 (P0_2)
- net FAULT_CRITICAL_SUM: now also TP2.1, U5.13 (P0_7)
- net FAULT_WARNING_SUM: now also U5.12 (P0_6)
- net GND: now also C1.2, C10.2, C12.2, C21.2, C22.2, C23.2, C30.2, C31.2, C32.2, C33.2, C36.1, C41.1, C49.1, C52.1, C6.2, C7.2, D11.1, D18.2, D3.1, J1.1, J2.1, J6.3 (Pin_3), J7.5 (Pin_5), R100.2, R13.2, R16.2, R17.1, R27.2, R29.2, R47.2, R54.2, R6.2, R65.2, R69.1, R78.2, R88.2, R97.2, U1.4 (GND), U1.4 (GND), U14.2 (GND), U15.2 (GND), U16.2 (GND), U3.4 (GND), U3.4 (GND), U5.18 (AD0), U5.24 (AD1), U5.25 (GND), U5.9 (GND), U8.3 (GND), U8.5 (~{ON}/OFF), U9.2 (GND); no longer C24.1
- net Gate _3.3_HIGH: now also D9.2 (cathode), Q7.4 (G), Q8.4 (G), R36.2, R92.2; no longer Q5.4 (G), R34.2
- net Gate _3.3_LOW: now also Q11.4 (G), D13.2 (cathode), R49.2, R98.2; no longer Q7.4 (G)
- net Gate _5_High: now also D2.2 (cathode), Q1.4 (G), Q2.4 (G), R75.2, R9.2; no longer D9.2 (cathode), Q11.4 (G), R23.2
- net Gate _5_LOW: now also Q5.4 (G), D6.2 (cathode), Q4.4 (G), R22.2, R82.2; no longer Q8.4 (G)
- net ISET_MPU_3V3: now also U5.11 (P0_5)
- net ISET_MPU_5V: now also U5.5 (P0_0)
- net I²C SCL_0: now also J6.2 (Pin_2), U5.19 (SCL)
- net I²C SDA_0: now also J6.1 (Pin_1), U5.20 (SDA)
- net SRC 3.3_HIGH: now also D9.1 (anode), Q7.1 (S), Q7.2 (S), Q7.3 (S), Q8.1 (S), Q8.2 (S), Q8.3 (S), R36.1, U15.8 (SRC); no longer Q5.1 (S), Q5.2 (S), Q5.3 (S)
- net SRC 3.3_LOW: now also Q11.1 (S), Q11.2 (S), Q11.3 (S), D13.1 (anode), R49.1, U16.8 (SRC); no longer Q7.1 (S), Q7.2 (S), Q7.3 (S)
- net SRC 5_HIGH: now also D2.1 (anode), Q1.1 (S), Q1.2 (S), Q1.3 (S), Q2.1 (S), Q2.2 (S), Q2.3 (S), R9.1, U9.8 (SRC); no longer D9.1 (anode), Q11.1 (S), Q11.2 (S), Q11.3 (S)
- net SRC 5_LOW: now also Q5.1 (S), Q5.2 (S), Q5.3 (S), D6.1 (anode), Q4.1 (S), Q4.2 (S), Q4.3 (S), R22.1, U14.8 (SRC); no longer Q8.1 (S), Q8.2 (S), Q8.3 (S)
- net VSENSE_3V3+: now also R27.1, R40.2, R41.2, U3.3
- net VSENSE_5V+: now also R12.2, R15.2, R6.1, U1.3
- net VSENSE_5V-: now also R17.2
- net V_out +3V3: now also L4.2, D12.2, J2.2, R41.1
- net V_out +5V: now also D4.2, J1.2, L1.2, R12.1; no longer L4.2
- net Ref_3.3V: now reaches C14.1, R32.2
- net Ref_3.3V: now also D8.3 (K)
- net at R34.1: now also C16.1, Q8.5 (D), R37.1
- net Ref_5V: now reaches C2.1, R3.2
- net Ref_5V: now also D1.3 (K)
- net at C16.2: now also C24.1, C22.1, C23.1, D11.2, R37.2, R38.1, R40.1, R46.1
- net at Q11.5 (D), R45.1, R51.1: now also C24.2
- net at R23.1: now also Q5.5 (D), C11.2, R19.1
- new net: R85.2, R88.1, U14.7 (OV)
- new net: C11.1, C3.2, C6.1, C7.1, D3.2, L1.1, R15.1, R19.2, R20.1, R7.2, R8.1
- new net: C3.1, Q2.5 (D), R4.1, R7.1
- new net: R43.1, U5.22 (~{INT})
- new net: C45.2, U14.4 (VCAP)
- new net: R82.1, U14.6 (GATE)
- new net: R28.2, R29.1, U3.5
- new net: D8.2 (A), U3.6, U3.7
- new net: R98.1, U16.6 (GATE)
- new net: D8.1 (A), U3.1, U3.2
- new net: R96.2, R97.1, U15.7 (OV)
- new net: D18.1, L5.1, U8.2 (OUT)
- new net: D12.1, R47.1
- new net: C51.2, U15.4 (VCAP)
- new net: R92.1, U15.6 (GATE)
- new net: D15.1, R54.1
- new net: D15.2, U5.1 (P1_0)
- new net: R42.1, U5.23 (~{RST})
- new net: C30.1, C31.1, R68.2, U8.1 (VIN)
- new net: C26.2, R61.1, R65.1, U8.4 (FB)
- new net: R100.1, R99.2, U16.7 (OV)
- new net: C38.2, U9.4 (VCAP)
- new net: R77.2, R78.1, U9.7 (OV)
- new net: R75.1, U9.6 (GATE)
- new net: D1.1 (A), U1.1, U1.2
- new net: D1.2 (A), U1.6, U1.7
- new net: R10.2, R13.1, U1.5
- new net: C53.2, U16.4 (VCAP)
- new net: D19.1, R69.2
- new net: D4.1, R16.1
- no-connect marks 10 -> 17
Other:
- note added: "3100 = 5.04V"
- note added: "Channel 1 Remote Sensing Network"
- note added: "Channel 2 Remote Sensing Network"
- note added: "Control Voltage Converter"
- moved on the sheet: C13, C14, C17, C18, C19, C2, C20, C25, C27, C28, C29, C34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
