File: hardware/kicad/dsp-regulator-rev-c/DSP-Regulator-RevC.kicad_sch (KiCad schematic)
At the start: 235 parts, among them J1 1935161, J2 1935161, J3 Wire con, J4 1935161, J5 Wire con, J6 Conn_01x03_Pin, J7 Conn_01x06_Pin, Q1 PSMN5R2-60YL, Q10 PSMN5R2-60YL, Q11 PSMN5R2-60YL, Q12 BSS138, Q2 PSMN5R2-60YL, Q3 BSS138, Q4 PSMN5R2-60YL, Q5 PSMN5R2-60YL, Q6 BSS138, Q7 PSMN5R2-60YL, Q8 PSMN5R2-60YL, Q9 BSS138, U1 TLV9352, U10 INA3221, U11 INA3221, U12 INA2180A2IDGKR, U13 TLV1702AIDGKR, U14 LM74502DDFR, U15 LM74502DDFR, U16 LM74502DDFR, U2 LM2596S-ADJ, U3 TLV9352, U4 LM2596S-ADJ, U5 AW9523B, U6 INA2180A2IDGKR, U7 TLV1702AIDGKR, U8 LM2596S-ADJ, U9 LM74502DDFR

Commit message: RB-013 LM74502 variant fix + Bucket 3 fault scope docs (salvaged)
Salvaged from phil-cia-bucket-3-execution-takeover, rebased onto current main.
Excludes the main.cpp Uart->HardwareSerial change, which would undo the
issue #3 build fix already on main.

Co-authored-by: Copilot App <223556219+Copilot@users.noreply.github.com>
Parts:
- U14, U15, U16, U9: value LM74502DDFR -> LM74502HDDFR
Changed lines of the file:
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@@
 			)
 		)
-		(property "Value" "LM74502DDFR"
+		(property "Value" "LM74502HDDFR"
 			(at 62.23 292.1 0)
 			(show_name no)
@@
 			)
 		)
-		(property "Value" "LM74502DDFR"
+		(property "Value" "LM74502HDDFR"
 			(at 62.23 335.28 0)
 			(show_name no)
@@
 			)
 		)
-		(property "Value" "LM74502DDFR"
+		(property "Value" "LM74502HDDFR"
 			(at 62.23 256.54 0)
 			(show_name no)
@@
 			)
 		)
-		(property "Value" "LM74502DDFR"
+		(property "Value" "LM74502HDDFR"
 			(at 62.23 370.84 0)
 			(show_name no)
