File: hardware/kicad/dsp-regulator-hat-rev-c/DSP-Regulator-HAT-RevC.kicad_sch (KiCad schematic)
At the start: 208 parts, among them J1 Conn_01x01_Pin, J10 USB Hub I2C, J11 SWD_Debug_Header, J12 FW-10-05-X-D-XXX-XXX-A, J13 Conn_01x01_Pin, J14 Conn_01x01_Pin, J15 Conn_01x01_Pin, J16 20021121-00010C4LF, J17 SWD_Debug_Header, J18 FW-10-05-X-D-XXX-XXX-A, J19 20021121-00010C4LF, J2 1935161, J3 Conn_01x01_Pin, J4 Conn_01x01_Pin, J5 1935161, J6 Conn_01x01_Pin, J7 Fan Control, J8 Connector, USB-TYPE-C-16P, J9 Display Uart, Q1 PSMN5R2-60YL, Q2 PSMN5R2-60YL, Q3 PSMN5R2-60YL, Q4 PSMN5R2-60YL, Q5 PSMN5R2-60YL, Q6 PSMN5R2-60YL, Q7 PSMN5R2-60YL, Q8 PSMN5R2-60YL, Q9 AO3400A, U1 LM74502HDDFR, U10 INA3221, U11 STM32_BLUE -, U12 W25Q128, U13 AHT20_C2757850, U14 74HC595D, U15 AMS1117-3.3, U16 CH340C, U2 INA2180A2IDGKR, U3 TLV1702AIDGKR, U4 LM74502HDDFR, U5 LM74502HDDFR, U6 INA2180A2IDGKR, U7 TLV1702AIDGKR, U8 LM74502HDDFR, U9 INA3221

Commit message: Update Rev-C regulator and HAT designs
Parts:
- removed C1, C10, C11, C12, C14, C16, C17, C20, C22, C23, C24, C25, C27, C28, C29, C3, C30, C31, C4, C8, C9: 100nF, PCM_JLCPCB:C_0805, symbol PCM_JLCPCB-Capacitors:0805,100nF,(2)
- removed C13, C15, C2, C26: 1nF, PCM_JLCPCB:C_0805, symbol PCM_JLCPCB-Capacitors:0805,1nF
- removed C18, C6: 470uf, Capacitor_SMD:CP_Elec_10x10, symbol Device:C_Small_US
- removed C19, C21, C5, C7: 10uF, PCM_JLCPCB:C_0805, symbol PCM_JLCPCB-Capacitors:0805,10uF,(2)
- removed D1, D6: 1N5819WS, Diode_SMD:D_SOD-323, symbol Diode:1N5819WS
- removed D10, D2, D5, D7: 1SMA4742A, PCM_JLCPCB:D_DO-214AC(SMA), symbol PCM_JLCPCB-Diodes:Zener,1SMA4742A
- removed D3, D8: SMBJ6.0CA, PCM_JLCPCB:D_SMB, symbol PCM_JLCPCB-Diodes:TVS-Bi,SMBJ6.0CA
- removed D4, D9: Green, PCM_JLCPCB:D_0805, symbol PCM_JLCPCB-Diodes:LED,0805,Green
- removed J1, J3, J4, J6: Conn_01x01_Pin, Connector_Wire:SolderWire-1sqmm_1x01_D1.4mm_OD2.7mm, symbol Connector:Conn_01x01_Pin
- removed J2, J5: 1935161, digikey-footprints:Terminal_Block_D1.3mm_P5mm, symbol dk_Terminal-Blocks-Wire-to-Board:1935161
- removed L1, L2: L_Ferrite, Inductor_SMD:L_1206_3216Metric, symbol Device:L_Ferrite
- removed POT1, POT2, POT3, POT4: 3296W-1-103LF, Potentiometer_THT:Potentiometer_Bourns_3296W_Vertical, symbol 1My_Basic components:3296W-1-103LF
- removed Q1, Q2, Q3, Q4, Q5, Q6, Q7, Q8: PSMN5R2-60YL, Package_TO_SOT_SMD:LFPAK56, symbol Transistor_FET:PSMN5R2-60YL
- removed R1, R12, R14, R22, R30, R32, R42, R46, R56, R61: 100kΩ, PCM_JLCPCB:R_0805, symbol PCM_JLCPCB-Resistors:0805,100kΩ
- removed R10, R23, R25, R27, R35, R37, R38, R5, R51, R54, R57, R9: 10kΩ, PCM_JLCPCB:R_0805, symbol PCM_JLCPCB-Resistors:0805,10kΩ
- removed R11, R16, R19, R20, R21, R24, R3, R34, R39, R4, R40, R45, R47, R49, R50, R53, R58, R8: 10Ω, PCM_JLCPCB:R_0805, symbol PCM_JLCPCB-Resistors:0805,10Ω
- removed R13, R15, R28, R29, R41, R43, R59, R60: 510kΩ, PCM_JLCPCB:R_0805, symbol PCM_JLCPCB-Resistors:0805,510kΩ
- removed R17, R48: 270Ω, PCM_JLCPCB:R_0805, symbol PCM_JLCPCB-Resistors:0805,270Ω
- removed R18: 200mΩ, Resistor_SMD:R_2512_6332Metric, symbol Device:R
- removed R2, R31, R33, R62: 1kΩ, PCM_JLCPCB:R_0805, symbol PCM_JLCPCB-Resistors:0805,1kΩ
- removed R26, R36, R55, R6: 390kΩ, PCM_JLCPCB:R_0805, symbol PCM_JLCPCB-Resistors:0805,390kΩ
- removed R44: 20m ohms, Resistor_SMD:R_2512_6332Metric, symbol Device:R
- removed R52: 200m ohms, Resistor_SMD:R_2512_6332Metric, symbol Device:R
- removed R7: 20mΩ, Resistor_SMD:R_2512_6332Metric, symbol Device:R
- removed TP1, TP2, TP3, TP4, TP5, TP6: TestPoint_Small, Connector_PinHeader_1.00mm:PinHeader_1x01_P1.00mm_Vertical, symbol Connector:TestPoint_Small
- removed U1, U4, U5, U8: LM74502HDDFR, Package_TO_SOT_SMD:Texas_DDF0008A_SOT-8_1.6x2.9mm_P0.65mm, symbol 1My_IC's:LM74502HDDFR
- removed U10, U9: INA3221, Package_DFN_QFN:Texas_RGV0016A_VQFN-16-1EP_4x4mm_P0.65mm_EP2.1x2.1mm, symbol Power_Management:INA3221
- removed U2, U6: INA2180A2IDGKR, Package_SO:VSSOP-8_3x3mm_P0.65mm, symbol Amplifier_Current:INA2180AxxDGK
- removed U3, U7: TLV1702AIDGKR, Package_SO:VSSOP-8_3x3mm_P0.65mm, symbol 1My_IC's:TLV1702AIDGKR
- added C43: 470uf 25V, Capacitor_SMD:CP_Elec_10x10.5, symbol Device:C_Polarized_US
- added C44, C47: 100nF, PCM_JLCPCB:C_0805, symbol PCM_JLCPCB-Capacitors:0805,100nF
- added C45: 100pF, PCM_JLCPCB:C_0805, symbol PCM_JLCPCB-Capacitors:0805,100pF
- added C46: 330uF 25v, Capacitor_SMD:CP_Elec_10x10.5, symbol Device:C_Polarized_US
- added D16: SS54B, PCM_JLCPCB:D_SMB, symbol PCM_JLCPCB-Diodes:Schottky,SS54B
- added D17: Yellow, PCM_JLCPCB:D_0805, symbol PCM_JLCPCB-Diodes_1:LED,0805,Yellow
- added L3: 33uh, Inductor_SMD:L_11.5x10mm_H6mm, symbol Device:L
- added R85: 0Ω, PCM_JLCPCB:R_1206, symbol PCM_JLCPCB-Resistors:1206,0Ω
- added R86: 1k, PCM_JLCPCB:R_0805, symbol PCM_JLCPCB-Resistors:0805,1kΩ
- added R87: 3100, PCM_JLCPCB:R_0805, symbol PCM_JLCPCB-Resistors:0805,100Ω
- added R88: 680Ω, PCM_JLCPCB:R_0805, symbol PCM_JLCPCB-Resistors:0805,680Ω
- added U17: LM2596S-ADJ, Package_TO_SOT_SMD:TO-263-5_TabPin3, symbol Regulator_Switching:LM2596S-ADJ
Connections:
- net +12V: now also R85.1
- net +5V_Boot: now also C45.1, C46.1, C47.1, D17.2, L3.2, R87.2
- net GND: now also C43.2, C44.2, C46.2, C47.2, D16.2, R86.2, R88.1, U17.3 (GND), U17.5 (~{ON}/OFF)
- new net: C43.1, C44.1, R85.2, U17.1 (VIN)
- new net: D16.1, L3.1, U17.2 (OUT)
- new net: C45.2, R86.1, R87.1, U17.4 (FB)
- new net: D17.1, R88.2
- no-connect marks 40 -> 30
Other:
- note added: "3100 = 5.04V"
- note added: "Control Voltage Converter"
- note removed: "Channel 1 5 volts"
- note removed: "Channel 2 3.3 volts"
- note removed: "Voltage Measuring"

Commit message: Update Rev-C coplanar board designs
Parts:
- removed C33: 100nF, PCM_JLCPCB:C_0805, symbol PCM_JLCPCB-Capacitors:0805,100nF,(2)
- removed C43: 470uf 25V, Capacitor_SMD:CP_Elec_10x10.5, symbol Device:C_Polarized_US
- removed C44, C47: 100nF, PCM_JLCPCB:C_0805, symbol PCM_JLCPCB-Capacitors:0805,100nF
- removed C45: 100pF, PCM_JLCPCB:C_0805, symbol PCM_JLCPCB-Capacitors:0805,100pF
- removed C46: 330uF 25v, Capacitor_SMD:CP_Elec_10x10.5, symbol Device:C_Polarized_US
- removed D13: Yellow, PCM_JLCPCB:D_0805, symbol PCM_JLCPCB-Diodes:LED,0805,Yellow
- removed D15: SMF05CT1G, PCM_JLCPCB:SOT-363_L2.0-W1.3-P0.65-LS2.1-BR, symbol PCM_JLCPCB-Diode-Packages:Package, SMF05CT1G
- removed D16: SS54B, PCM_JLCPCB:D_SMB, symbol PCM_JLCPCB-Diodes:Schottky,SS54B
- removed D17: Yellow, PCM_JLCPCB:D_0805, symbol PCM_JLCPCB-Diodes_1:LED,0805,Yellow
- removed J16: 20021121-00010C4LF, digikey-footprints:PinHeader_2x5_P1.27mm, symbol 1My_Basic components:20021121-00010C4LF
- removed L3: 33uh, Inductor_SMD:L_11.5x10mm_H6mm, symbol Device:L
- removed R71: 10kΩ, PCM_JLCPCB:R_0805, symbol PCM_JLCPCB-Resistors:0805,10kΩ
- removed R72: 270Ω, PCM_JLCPCB:R_0805, symbol PCM_JLCPCB-Resistors:0805,270Ω
- removed R85: 0Ω, PCM_JLCPCB:R_1206, symbol PCM_JLCPCB-Resistors:1206,0Ω
- removed R86: 1k, PCM_JLCPCB:R_0805, symbol PCM_JLCPCB-Resistors:0805,1kΩ
- removed R87: 3100, PCM_JLCPCB:R_0805, symbol PCM_JLCPCB-Resistors:0805,100Ω
- removed R88: 680Ω, PCM_JLCPCB:R_0805, symbol PCM_JLCPCB-Resistors:0805,680Ω
- removed U14: 74HC595D, PCM_JLCPCB:SOIC-16_L9.9-W3.9-P1.27-LS6.0-BL, symbol PCM_JLCPCB-ICs:Shift Register, 1 In, 8 Out, 74HC595D,118
- removed U17: LM2596S-ADJ, Package_TO_SOT_SMD:TO-263-5_TabPin3, symbol Regulator_Switching:LM2596S-ADJ
- added C57: 100nF, PCM_JLCPCB:C_0805, symbol PCM_JLCPCB-Capacitors:0805,100nF
- added U2: ESP32_C3_mini, 113991054:MODULE_113991054, symbol 1My_MPUs:ESP32_C3_mini
- C34, C35, D11, J7, Q9, R63, R64, R67, R68, U12: now not fitted
Connections:
- net +5V_Boot: now also C57.1, U2.16 (5V)
- net FAULT_CRITICAL_SUM: no longer U11.28 (A3)
- net FAULT_WARNING_SUM: no longer U11.33 (B0)
- net GND: now also C57.2, U2.15 (GND)
- net TXD_ESP: now reaches U11.27 (A2)
- net TXD_ESP: now also U2.10 (GPIO1)
- new net CTS_ESP: U2.7 (GPIO20)
- new net RTS_ESP: U2.8 (GPIO21)
- new net RXD_ESP: U11.28 (A3), U2.9 (GPIO0)
- no-connect marks 30 -> 37
Other:
- note added: "RX-1"
- note added: "RX-2"
- note added: "RX-3"
- note added: "TX-1"
- note added: "TX-2"
- note added: "TX-3"
- note removed: "3100 = 5.04V"
- note removed: "Control Voltage Converter"
- note removed: "Logic analyzer connector"
- note removed: "Regulator control outputs"
- moved on the sheet: H1, H2, H3, H4, J13, J14, J15
