File: hardware/kicad/dsp-regulator-hat-rev-d-full/MCU.kicad_sch (KiCad schematic)
At the start: 31 parts, among them J1 ARM 10-pin keyed SWD header (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, J2 BOOT0 recovery jumper (fit to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, J3 GCT USB4105-GF-A, J4 ESP32-C3-MINI-1U interface (e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, SW1 RESET, U1 STM32F405RGT6, U2 USBLC6-2SC6, Y1 8.000MHz (candidate; UNVERIFI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

Commit message: hw(hat): start source-backed Rev-D HAT integration
Import an independent HAT reuse sheet, replace legacy controller endpoints with frozen F405 interfaces and reset biases, and record partial-integration gaps and unresolved inherited ERC warnings. Support-only and Rev-C sources remain byte-identical; no PCB or bench validation claimed.

Co-authored-by: Copilot App <223556219+Copilot@users.noreply.github.com>
Parts:
- added R11, R12, R15, R16, R17, R18, R19: 10k, Resistor_SMD:R_0603_1608Metric, symbol Device:R
- added R13, R14: 47k, Resistor_SMD:R_0603_1608Metric, symbol Device:R
Connections:
- net +3V3: now also R15.1, R16.1, R17.1, R18.1, R19.1
- net GND: now also R11.2, R12.2, R13.2, R14.2
- net ISET_MPU_5V: now reaches U1.14 (PA0)
- net ISET_MPU_5V: now also R11.1
- net ISET_MPU_3V3: now reaches U1.15 (PA1)
- net ISET_MPU_3V3: now also R12.1
- net SPI_SCK: now reaches U1.21 (PA5)
- net SPI_SCK: now also R13.1
- net SPI_MISO: now reaches U1.22 (PA6)
- net SPI_MOSI: now reaches U1.23 (PA7)
- net SPI_MOSI: now also R14.1
- net DISP_UART_TX: now reaches U1.29 (PB10)
- net DISP_UART_TX: now also R18.2
- net DISP_UART_RX: now reaches U1.30 (PB11)
- net DISP_UART_RX: now also R19.2
- net Memory_CS: now reaches U1.41 (PA8)
- net Memory_CS: now also R15.2
- net FAN_PWM: now reaches U1.57 (PB5)
- net UART1_TX: now reaches U1.58 (PB6)
- net UART1_TX: now also R16.2
- net UART1_RX: now reaches U1.59 (PB7)
- net UART1_RX: now also R17.2
- net I²C SCL_0: now reaches U1.61 (PB8)
- net I²C SDA_0: now reaches U1.62 (PB9)
- no-connect marks 44 -> 31
Other:
- note added: "Frozen interface biases added for first-pass reuse. PA4/PC4/PC13 remain NC: source-backed endpoints/replacements still pending. C3 J4 remains logical only; bare module integration pending."
